Commit message: [kinikun] add script to add exramodule, rename quadrotor to kinikun in launch

File: robots/kinikun/urdf/robot.gazebo.xacro (robot description, xacro)
@@ -2,5 +2,5 @@
 <robot
     xmlns:xacro="http://www.ros.org/wiki/xacro" name="kinikun" >
-  <xacro:arg name="robot_name" default="quadrotor" />
+  <xacro:arg name="robot_name" default="kinikun" />
   <!-- robot urdf -->
   <xacro:include filename="$(find kinikun)/urdf/robot.urdf.xacro" />

File: robots/kinikun/urdf/robot.urdf.xacro (robot description, xacro)
@@ -1,5 +1,5 @@
 <?xml version="1.0"?>
 <robot
-    xmlns:xacro="http://www.ros.org/wiki/xacro" name="module_quadrotor" >
+  xmlns:xacro="http://www.ros.org/wiki/xacro" name="module_quadrotor">
   <!-- general attribute -->
   <baselink name="fc" />
@@ -19,8 +19,9 @@
     </gazebo>
   </xacro:macro>
-  <xacro:macro name="extra_module" params="name parent *origin *inertial visible:=0 model_url:=1 scale:=1">
+  <xacro:macro name="extra_module"
+    params="name parent *origin *inertial visible:=0 model_url:=1 scale:=1">
     <joint name="${parent}2${name}" type="fixed">
-      <parent link="${parent}"/>
-      <child link="${name}"/>
+      <parent link="${parent}" />
+      <child link="${name}" />
       <xacro:insert_block name="origin" />
     </joint>
@@ -29,7 +30,7 @@
       <xacro:if value="${visible == 1}">
         <visual>
-          <origin rpy="0 0 0" xyz="0 0 0"/>
+          <origin rpy="0 0 0" xyz="0 0 0" />
           <geometry>
-            <mesh filename="${model_url}" scale= "${scale} ${scale} ${scale}"/>
+            <mesh filename="${model_url}" scale="${scale} ${scale} ${scale}" />
           </geometry>
         </visual>
@@ -37,72 +38,33 @@
     </link>
   </xacro:macro>
-  <xacro:macro name="propeller_module" params="id x y z direction">
-    <joint name="rotor${id}" type="continuous">
-      <limit effort="100.0" lower="${min_force}" upper="${max_force}" velocity="0.5"/>
-      <parent link="main_body"/>
-      <child link="thrust${id}"/>
-      <origin rpy="0 0 0" xyz="${x} ${y} ${z}"/>
-      <axis xyz="0 0 ${direction}"/>
-    </joint>
-    <link name="thrust${id}">
-      <!-- visual & collisiont -->
-      <inertial>
-        <origin xyz="0 0 0" rpy="0 0 0"/>
-        <mass value="0.0091"/>
-        <inertia
-            ixx="0.00000807" ixy="0.0" ixz="0.0"
-            iyy="0.00000807" iyz="0.0"
-            izz="0.00001612"/>
-      </inertial>
-      <visual>
-        <origin rpy="0 0 0" xyz="0 0 0"/>
-        <geometry>
-          <mesh filename="package://kinikun/urdf/mesh/prop_5inch.dae" />
-        </geometry>
-      </visual>
-    </link>
-    <xacro:damping_factor link ="thrust${id}"/>
-    <transmission name="rotor_tran${id}">
-      <type>transmission_interface/SimpleTransmission</type>
-      <joint name="rotor${id}">
-        <!-- TODO: effort is torque, maybe position is enough -->
-        <hardwareInterface>RotorInterface</hardwareInterface>
-      </joint>
-      <actuator name="rotor${id}">
-        <!-- TODO: effort is torque, maybe position is enough -->
-        <hardwareInterface>RotorInterface</hardwareInterface>
-        <mechanicalReduction>1</mechanicalReduction>
-      </actuator>
-    </transmission>
-  </xacro:macro>
   <!-- dummy root link for KDL -->
   <link name="root">
     <inertial>
-      <origin xyz="0 0 0" rpy="0 0 0"/>
-      <mass value="0.00001"/>
-      <inertia
-          ixx="0.000001" ixy="0.0" ixz="0.0"
-          iyy="0.000001" iyz="0.0"
-          izz="0.000002"/>
+      <origin xyz="0 0 0" rpy="0 0 0" />
+      <mass value="0.00001" />
+      <inertia
+        ixx="0.000001" ixy="0.0" ixz="0.0"
+        iyy="0.000001" iyz="0.0"
+        izz="0.000002" />
     </inertial>
   </link>
   <joint name="root_joint" type="fixed">
-    <parent link="root"/>
-    <child link="main_body"/>
-    <origin rpy="0 0 0" xyz="0 0 0"/>
-    <axis xyz="0 0 1"/>
+    <parent link="root" />
+    <child link="main_body" />
+    <origin rpy="0 0 0" xyz="0 0 0" />
+    <axis xyz="0 0 1" />
   </joint>
   <!-- main_body -->
   <link name="main_body">
     <inertial>
-      <mass value = "0.276" />
-      <origin xyz="0 0 0.017" rpy="0 0 0"/>
-      <inertia
-          ixx="0.0021" ixy="0" ixz="0"
-          iyy="0.0015" iyz="0"
-          izz="0.0032"/>
-    </inertial>
-    <visual>
-      <origin rpy="0 0 0" xyz="0 0 0"/>
+      <mass value="0.276" />
+      <origin xyz="0 0 0.017" rpy="0 0 0" />
+      <inertia
+        ixx="0.0021" ixy="0" ixz="0"
+        iyy="0.0015" iyz="0"
+        izz="0.0032" />
+    </inertial>
+    <visual>
+      <origin rpy="0 0 0" xyz="0 0 0" />
       <geometry>
         <mesh filename="package://kinikun/urdf/mesh/main_body.dae" />
@@ -110,5 +72,5 @@
     </visual>
     <collision>
-      <origin rpy="0 0 0" xyz="0 0 0"/>
+      <origin rpy="0 0 0" xyz="0 0 0" />
       <geometry>
         <box size="0.28 0.28 0.072" />
@@ -117,297 +79,404 @@
   </link>
   <!-- spinal -->
-  <xacro:extra_module name = "fc" parent = "main_body" visible = "0" >
-    <origin xyz="0 0 0" rpy="0 0 0"/>
-    <inertial>
-      <mass value = "00" />
-      <origin xyz="0 0 0" rpy="0 0 0"/>
-      <inertia
-          ixx="0.0" ixy="0.0" ixz="0.0"
-          iyy="0.0" iyz="0.0" izz="0.0"/>
+  <xacro:extra_module name="fc" parent="main_body" visible="0">
+    <origin xyz="0 0 0" rpy="0 0 0" />
+    <inertial>
+      <mass value="00" />
+      <origin xyz="0 0 0" rpy="0 0 0" />
+      <inertia
+        ixx="0.0" ixy="0.0" ixz="0.0"
+        iyy="0.0" iyz="0.0" izz="0.0" />
     </inertial>
   </xacro:extra_module>
   <!-- battery -->
-  <xacro:extra_module name = "battery" parent = "main_body" visible = "1" model_url = "package://kinikun/urdf/mesh/turnigy_3S_2200mAh.dae" >
-    <origin xyz="0.0105 0 -0.012" rpy="0 0 0"/>
-    <inertial>
-      <mass value = "0.188" />
-      <origin xyz="0 0 0" rpy="0 0 0"/>
-      <inertia
-          ixx="0.0002" ixy="0.0" ixz="0.0"
-          iyy="0.0002" iyz="0.0" izz="0.0002"/>
+  <xacro:extra_module name="battery" parent="main_body" visible="1"
+    model_url="package://kinikun/urdf/mesh/turnigy_3S_2200mAh.dae">
+    <origin xyz="0.0105 0 -0.012" rpy="0 0 0" />
+    <inertial>
+      <mass value="0.188" />
+      <origin xyz="0 0 0" rpy="0 0 0" />
+      <inertia
+        ixx="0.0002" ixy="0.0" ixz="0.0"
+        iyy="0.0002" iyz="0.0" izz="0.0002" />
     </inertial>
   </xacro:extra_module>
-  <!-- propellers -->
-  <!-- <xacro:propeller_module id = "1" x = "${-rotor_x}" y = "${-rotor_y}" z = "${rotor_z}" direction = "-1" /> -->
-  <!-- <xacro:propeller_module id = "2" x = "${rotor_x}" y = "${-rotor_y}" z = "${rotor_z}" direction = "1" />
-  <xacro:propeller_module id = "3" x = "${rotor_x}" y = "${rotor_y}" z = "${rotor_z}" direction = "-1" />
-  <xacro:propeller_module id = "4" x = "${-rotor_x}" y = "${rotor_y}" z = "${rotor_z}"  direction = "1" /> -->
- <joint name="arm1_joint" type="fixed">
+  <joint name="arm1_joint" type="fixed">
     <!-- <limit lower="${-pi/4}" upper="${pi/4}" effort="10.0" velocity="0.5"/> -->
-    <parent link="main_body"/>
-    <child link="arm1_link"/>
-    <origin xyz="-0.03 -0.03 0" rpy="0 0 ${ -3*pi / 4}"/>
-    <axis xyz="0 0 1"/>
-    <dynamics damping="0.9" friction="0.05"/>
+    <parent link="main_body" />
+    <child link="arm1_link" />
+    <origin xyz="-0.03 -0.03 0" rpy="0 0 ${ -3*pi / 4}" />
+    <axis xyz="0 0 1" />
+    <dynamics damping="0.9" friction="0.05" />
   </joint>
   <link name="arm1_link">
-    <origin xyz="0 0 0" rpy="0 0 0"/>
-    <inertial>
-      <origin xyz="${0.21 / 2 - 0.004} 0 0" rpy="0 0 0"/>
-      <mass value="0.12"/>
+    <origin xyz="0 0 0" rpy="0 0 0" />
+    <inertial>
+      <origin xyz="${0.21 / 2 - 0.004} 0 0" rpy="0 0 0" />
+      <mass value="0.12" />
       <inertia
         ixx="0.001804" iyy="0.017972" izz="0.019248"
-        ixy="0.000021" ixz="0.000372" iyz="0.000000"/>
-    </inertial>
-    <visual>
-      <origin xyz="${0.21 / 2 - 0.004} 0 0" rpy="0 0 0"/>
-      <geometry>
-  <box size="0.21 0.015 0.005"/>
-      </geometry>
-    </visual>
-  </link>
- <joint name="rotor1" type="continuous">
-   <parent link="arm1_link"/>
-   <child link="thrust1"/>
-   <origin xyz="0.19 0 0 " rpy="0 0 0"/>
-   <axis xyz="0 0 -1"/>
-   <limit effort="100" lower="${min_force}" upper="${max_force}" velocity="0.5"/>
+        ixy="0.000021" ixz="0.000372" iyz="0.000000" />
+    </inertial>
+    <visual>
+      <origin xyz="${0.21 / 2 - 0.004} 0 0" rpy="0 0 0" />
+      <geometry>
+        <box size="0.21 0.015 0.005" />
+      </geometry>
+    </visual>
+  </link>
+  <joint name="rotor1" type="continuous">
+    <parent link="arm1_link" />
+    <child link="thrust1" />
+    <origin xyz="0.19 0 0 " rpy="0 0 0" />
+    <axis xyz="0 0 -1" />
+    <limit effort="100" lower="${min_force}" upper="${max_force}" velocity="0.5" />
   </joint>
   <link name="thrust1">
-      <!-- visual & collisiont -->
-      <inertial>
-        <origin xyz="0 0 0" rpy="0 0 0"/>
-        <mass value="0.0091"/>
-        <inertia
-            ixx="0.00000807" ixy="0.0" ixz="0.0"
-            iyy="0.00000807" iyz="0.0"
-            izz="0.00001612"/>
-      </inertial>
-      <visual>
-        <origin rpy="0 0 0" xyz="0 0 0"/>
-        <geometry>
-          <mesh filename="package://kinikun/urdf/mesh/prop_5inch.dae" />
-        </geometry>
-      </visual>
-    </link>
-    <xacro:damping_factor link ="thrust1"/>
-    <transmission name="rotor_tran1">
-      <type>transmission_interface/SimpleTransmission</type>
-      <joint name="rotor1">
-        <!-- TODO: effort is torque, maybe position is enough -->
-        <hardwareInterface>RotorInterface</hardwareInterface>
-      </joint>
-      <actuator name="rotor1">
-        <!-- TODO: effort is torque, maybe position is enough -->
-        <hardwareInterface>RotorInterface</hardwareInterface>
-        <mechanicalReduction>1</mechanicalReduction>
-      </actuator>
-    </transmission>
-<joint name="arm2_joint" type="revolute">
-    <limit lower="${-pi/4}" upper="${pi/4}" effort="10.0" velocity="0.5"/>
-    <parent link="main_body"/>
-    <child link="arm2_link"/>
-    <origin xyz="0.03 -0.03 0" rpy="0 0 ${- pi / 4}"/>
-    <axis xyz="0 0 1"/>
-    <dynamics damping="0.9" friction="0.05"/>
+    <!-- visual & collisiont -->
+    <inertial>
+      <origin xyz="0 0 0" rpy="0 0 0" />
+      <mass value="0.0091" />
+      <inertia
+        ixx="0.00000807" ixy="0.0" ixz="0.0"
+        iyy="0.00000807" iyz="0.0"
+        izz="0.00001612" />
+    </inertial>
+    <visual>
+      <origin rpy="0 0 0" xyz="0 0 0" />
+      <geometry>
+        <mesh filename="package://kinikun/urdf/mesh/prop_5inch.dae" />
+      </geometry>
+    </visual>
+  </link>
+  <xacro:damping_factor link="thrust1" />
+  <transmission name="rotor_tran1">
+    <type>transmission_interface/SimpleTransmission</type>
+    <joint name="rotor1">
+      <!-- TODO: effort is torque, maybe position is enough -->
+      <hardwareInterface>RotorInterface</hardwareInterface>
+    </joint>
+    <actuator name="rotor1">
+      <!-- TODO: effort is torque, maybe position is enough -->
+      <hardwareInterface>RotorInterface</hardwareInterface>
+      <mechanicalReduction>1</mechanicalReduction>
+    </actuator>
+  </transmission>
+  <joint name="arm2_joint" type="revolute">
+    <limit lower="${-pi/4}" upper="${pi/4}" effort="10.0" velocity="0.5" />
+    <parent link="main_body" />
+    <child link="arm2_link" />
+    <origin xyz="0.03 -0.03 0" rpy="0 0 ${- pi / 4}" />
+    <axis xyz="0 0 1" />
+    <dynamics damping="0.9" friction="0.05" />
   </joint>
   <link name="arm2_link">
-    <origin xyz="0 0 0" rpy="0 0 0"/>
-    <inertial>
-      <origin xyz="${0.21 / 2 - 0.004} 0 0" rpy="0 0 0"/>
-      <mass value="0.200"/>
+    <origin xyz="0 0 0" rpy="0 0 0" />
+    <inertial>
+      <origin xyz="${0.21 / 2 - 0.004} 0 0" rpy="0 0 0" />
+      <mass value="0.200" />
       <inertia
         ixx="0.001804" iyy="0.017972" izz="0.019248"
-        ixy="0.000021" ixz="0.000372" iyz="0.000000"/>
-    </inertial>
-    <visual>
-      <origin xyz="${0.21 / 2 - 0.004} 0 0" rpy="0 0 0"/>
-      <geometry>
-  <box size="0.21 0.015 0.005"/>
-      </geometry>
-    </visual>
-  </link>
- <joint name="rotor2" type="continuous">
-   <parent link="arm2_link"/>
-   <child link="thrust2"/>
-   <origin xyz="0.19 0 0 " rpy="0 0 0"/>
-   <axis xyz="0 0 1"/>
-   <limit effort="100" lower="${min_force}" upper="${max_force}" velocity="0.5"/>
+        ixy="0.000021" ixz="0.000372" iyz="0.000000" />
+    </inertial>
+    <visual>
+      <origin xyz="${0.21 / 2 - 0.004} 0 0" rpy="0 0 0" />
+      <geometry>
+        <box size="0.21 0.015 0.005" />
+      </geometry>
+    </visual>
+  </link>
+  <joint name="rotor2" type="continuous">
+    <parent link="arm2_link" />
+    <child link="thrust2" />
+    <origin xyz="0.19 0 0 " rpy="0 0 0" />
+    <axis xyz="0 0 1" />
+    <limit effort="100" lower="${min_force}" upper="${max_force}" velocity="0.5" />
   </joint>
   <link name="thrust2">
-      <!-- visual & collisiont -->
-      <inertial>
-        <origin xyz="0 0 0" rpy="0 0 0"/>
-        <mass value="0.0091"/>
-        <inertia
-            ixx="0.00000807" ixy="0.0" ixz="0.0"
-            iyy="0.00000807" iyz="0.0"
-            izz="0.00001612"/>
-      </inertial>
-      <visual>
-        <origin rpy="0 0 0" xyz="0 0 0"/>
-        <geometry>
-          <mesh filename="package://kinikun/urdf/mesh/prop_5inch.dae" />
-        </geometry>
-      </visual>
-    </link>
-    <xacro:damping_factor link ="thrust2"/>
-    <transmission name="rotor_tran2">
-      <type>transmission_interface/SimpleTransmission</type>
-      <joint name="rotor2">
-        <!-- TODO: effort is torque, maybe position is enough -->
-        <hardwareInterface>RotorInterface</hardwareInterface>
-      </joint>
-      <actuator name="rotor2">
-        <!-- TODO: effort is torque, maybe position is enough -->
-        <hardwareInterface>RotorInterface</hardwareInterface>
-        <mechanicalReduction>1</mechanicalReduction>
-      </actuator>
-    </transmission>
-        <transmission name="joint_tran2">
-        <type>transmission_interface/SimpleTransmission</type>
-        <joint name="arm2_joint">
-          <!-- TODO: effort is torque, maybe position is enough -->
-          <hardwareInterface>hardware_interface/EffortJointInterface</hardwareInterface>
-        </joint>
-        <actuator name="servo2">
-          <!-- TODO: effort is torque, maybe position is enough -->
-          <hardwareInterface>hardware_interface/EffortJointInterface</hardwareInterface>
-          <mechanicalReduction>1</mechanicalReduction>
-        </actuator>
-    </transmission>
- <joint name="arm3_joint" type="revolute">
-    <limit lower="${-pi/3}" upper="${pi/3}" effort="10.0" velocity="0.5"/>
-    <parent link="main_body"/>
-    <child link="arm3_link"/>
-    <origin xyz="0.03 0.03 0" rpy="0 0 ${ pi / 4}"/>
-    <axis xyz="0 0 1"/>
-    <dynamics damping="0.9" friction="0.05"/>
+    <!-- visual & collisiont -->
+    <inertial>
+      <origin xyz="0 0 0" rpy="0 0 0" />
+      <mass value="0.0091" />
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