Commit message: [kinikun] add kinikun2 urdf and modify inertia of arm link

File: robots/kinikun/urdf/robot.gazebo.xacro (robot description, xacro)
@@ -4,5 +4,5 @@
   <xacro:arg name="robot_name" default="kinikun" />
   <!-- robot urdf -->
-  <xacro:include filename="$(find kinikun)/urdf/robot.urdf.xacro" />
+  <xacro:include filename="$(find kinikun)/urdf/robot2.urdf.xacro" />
   <!-- gazebo plugin for default controller and sensors -->
   <xacro:include filename="$(find aerial_robot_simulation)/xacro/spinal.gazebo.xacro" />

File: robots/kinikun/urdf/robot.urdf.xacro (robot description, xacro)
@@ -68,5 +68,5 @@
       <origin rpy="0 0 0" xyz="0 0 0" />
       <geometry>
-        <mesh filename="package://kinikun/urdf/mesh/kinikun_main_body.dae" />
+        <mesh filename="package://kinikun/urdf/mesh/kinikun/kinikun_main_body.dae" />
       </geometry>
     </visual>
@@ -121,5 +121,5 @@
       <origin xyz="0 0 0" rpy="0 0 0" />
       <geometry>
-        <mesh filename="package://kinikun/urdf/mesh/kinikun_foot_R.dae" />
+        <mesh filename="package://kinikun/urdf/mesh/kinikun/kinikun_foot_R.dae" />
       </geometry>
     </visual>
@@ -183,5 +183,5 @@
       <origin xyz="0 0 0" rpy="0 0 0" />
       <geometry>
-        <mesh filename="package://kinikun/urdf/mesh/kinikun_foot_L.dae" />
+        <mesh filename="package://kinikun/urdf/mesh/kinikun/kinikun_foot_L.dae" />
       </geometry>
     </visual>
@@ -256,5 +256,5 @@
       <origin xyz="0 0 0" rpy="0 0 0" />
       <geometry>
-        <mesh filename="package://kinikun/urdf/mesh/kinikun_foot_R.dae" />
+        <mesh filename="package://kinikun/urdf/mesh/kinikun/kinikun_foot_R.dae" />
       </geometry>
     </visual>
@@ -329,5 +329,5 @@
       <origin xyz="0 0 0" rpy="0 0 0" />
       <geometry>
-        <mesh filename="package://kinikun/urdf/mesh/kinikun_foot_L.dae" />
+        <mesh filename="package://kinikun/urdf/mesh/kinikun/kinikun_foot_L.dae" />
       </geometry>
     </visual>

File: robots/kinikun/urdf/robot2.urdf.xacro (robot description, xacro)
@@ -58,21 +58,21 @@
   <link name="main_body">
     <inertial>
-      <mass value="0.276" />
-      <origin xyz="0 0 0.017" rpy="0 0 0" />
+      <mass value="0.239" />
+      <origin xyz="0 0 0.064" rpy="0 0 0" />
       <inertia
         ixx="0.0021" ixy="0" ixz="0"
         iyy="0.0015" iyz="0"
-        izz="0.0032" />
-    </inertial>
-    <visual>
-      <origin rpy="0 0 0" xyz="0 0 0" />
-      <geometry>
-        <mesh filename="package://kinikun/urdf/mesh/main_body.dae" />
+        izz="0.0032"/>
+    </inertial>
+    <visual>
+      <origin rpy="0 0 0" xyz="0 0 0.080" />
+      <geometry>
+        <mesh filename="package://kinikun/urdf/mesh/kinikun2/main_body.dae" />
       </geometry>
     </visual>
     <collision>
-      <origin rpy="0 0 0" xyz="0 0 0" />
-      <geometry>
-        <box size="0.28 0.28 0.072" />
+      <origin rpy="0 0 0" xyz="0 0 0.064" />
+      <geometry>
+        <box size="0.1 0.1 0.018" />
       </geometry>
     </collision>
@@ -82,5 +82,5 @@
     <origin xyz="0 0 0" rpy="0 0 0" />
     <inertial>
-      <mass value="00" />
+      <mass value="0.0" />
       <origin xyz="0 0 0" rpy="0 0 0" />
       <inertia
@@ -89,5 +89,5 @@
     </inertial>
   </xacro:extra_module>
-  <!-- battery -->
+  <!-- battery
   <xacro:extra_module name="battery" parent="main_body" visible="1"
     model_url="package://kinikun/urdf/mesh/turnigy_3S_2200mAh.dae">
@@ -100,35 +100,25 @@
         iyy="0.0002" iyz="0.0" izz="0.0002" />
     </inertial>
-  </xacro:extra_module>
-  <!-- propellers -->
-  <!-- <xacro:propeller_module id = "1" x = "${-rotor_x}" y = "${-rotor_y}" z = "${rotor_z}"
-  direction = "-1" /> -->
-  <!-- <xacro:propeller_module id = "2" x = "${rotor_x}" y = "${-rotor_y}" z = "${rotor_z}"
-  direction = "1" />
-  <xacro:propeller_module id = "3" x = "${rotor_x}" y = "${rotor_y}" z = "${rotor_z}" direction =
-  "-1" />
-  <xacro:propeller_module id = "4" x = "${-rotor_x}" y = "${rotor_y}" z = "${rotor_z}"  direction =
-  "1" /> -->
-  <joint name="arm1_joint" type="fixed">
-    <!-- <limit lower="${-pi/4}" upper="${pi/4}" effort="10.0" velocity="0.5"/> -->
+  </xacro:extra_module> -->
+  <joint name="arm1_joint" type="revolute">
+    <limit lower="${-pi/4}" upper="${pi/4}" effort="1.0" velocity="0.5"/>
     <parent link="main_body" />
     <child link="arm1_link" />
-    <origin xyz="-0.03 -0.03 0" rpy="0 0 ${ -3*pi / 4}" />
+    <origin xyz="-0.03015 -0.03015 0.06938" rpy="0 0 ${ -3*pi / 4}" />
     <axis xyz="0 0 1" />
     <dynamics damping="0.9" friction="0.05" />
   </joint>
   <link name="arm1_link">
-    <origin xyz="0 0 0" rpy="0 0 0" />
-    <inertial>
-      <origin xyz="${0.21 / 2 - 0.004} 0 0" rpy="0 0 0" />
-      <mass value="0.12" />
+    <inertial>
+      <origin xyz="0.138 0 -0.00104" rpy="0 0 0" />
+      <mass value="0.191" />
       <inertia
         ixx="0.001804" iyy="0.017972" izz="0.019248"
-        ixy="0.000021" ixz="0.000372" iyz="0.000000" />
-    </inertial>
-    <visual>
-      <origin xyz="${0.21 / 2 - 0.004} 0 0" rpy="0 0 0" />
-      <geometry>
-        <box size="0.21 0.015 0.005" />
+        ixy="0.000021" ixz="0.000372" iyz="0.000000"/>
+    </inertial>
+    <visual>
+      <origin xyz="0.138 0 -0.00104" rpy="0 0 0" />
+      <geometry>
+        <mesh filename="package://kinikun/urdf/mesh/kinikun2/arm.dae" />
       </geometry>
     </visual>
@@ -137,5 +127,5 @@
     <parent link="arm1_link" />
     <child link="thrust1" />
-    <origin xyz="0.19 0 0 " rpy="0 0 0" />
+    <origin xyz="0.179 0 0.0209" rpy="0 0 0" />
     <axis xyz="0 0 -1" />
     <limit effort="100" lower="${min_force}" upper="${max_force}" velocity="0.5" />
@@ -171,25 +161,36 @@
     </actuator>
   </transmission>
+      <transmission name="joint_tran1">
+      <type>transmission_interface/SimpleTransmission</type>
+      <joint name="arm1_joint">
+        <!-- TODO: effort is torque, maybe position is enough -->
+        <hardwareInterface>hardware_interface/EffortJointInterface</hardwareInterface>
+      </joint>
+      <actuator name="servo1">
+        <!-- TODO: effort is torque, maybe position is enough -->
+        <hardwareInterface>hardware_interface/EffortJointInterface</hardwareInterface>
+        <mechanicalReduction>1</mechanicalReduction>
+      </actuator>
+  </transmission>
   <joint name="arm2_joint" type="revolute">
-    <limit lower="${-pi/4}" upper="${pi/4}" effort="10.0" velocity="0.5" />
+    <limit lower="${-pi/4}" upper="${pi/4}" effort="1.0" velocity="0.5" />
     <parent link="main_body" />
     <child link="arm2_link" />
-    <origin xyz="0.03 -0.03 0" rpy="0 0 ${- pi / 4}" />
+    <origin xyz="0.03015 -0.03015 0.06938" rpy="0 0 ${- pi / 4}" />
     <axis xyz="0 0 1" />
     <dynamics damping="0.9" friction="0.05" />
   </joint>
   <link name="arm2_link">
-    <origin xyz="0 0 0" rpy="0 0 0" />
-    <inertial>
-      <origin xyz="${0.21 / 2 - 0.004} 0 0" rpy="0 0 0" />
-      <mass value="0.200" />
+    <inertial>
+      <origin xyz="0.138 0 -0.00104" rpy="0 0 0" />
+      <mass value="0.191" />
       <inertia
         ixx="0.001804" iyy="0.017972" izz="0.019248"
-        ixy="0.000021" ixz="0.000372" iyz="0.000000" />
-    </inertial>
-    <visual>
-      <origin xyz="${0.21 / 2 - 0.004} 0 0" rpy="0 0 0" />
-      <geometry>
-        <box size="0.21 0.015 0.005" />
+        ixy="0.000021" ixz="0.000372" iyz="0.000000"/>
+    </inertial>
+    <visual>
+      <origin xyz="0.138 0 -0.00104" rpy="0 0 0" />
+      <geometry>
+        <mesh filename="package://kinikun/urdf/mesh/kinikun2/arm.dae" />
       </geometry>
     </visual>
@@ -198,5 +199,5 @@
     <parent link="arm2_link" />
     <child link="thrust2" />
-    <origin xyz="0.19 0 0 " rpy="0 0 0" />
+    <origin xyz="0.179 0 0.0209" rpy="0 0 0" />
     <axis xyz="0 0 1" />
     <limit effort="100" lower="${min_force}" upper="${max_force}" velocity="0.5" />
@@ -219,5 +220,5 @@
     </visual>
   </link>
-  <xacro:damping_factor link="thrust2" />
+  <xacro:damping_factor link ="thrust2"/>
   <transmission name="rotor_tran2">
     <type>transmission_interface/SimpleTransmission</type>
@@ -233,36 +234,35 @@
   </transmission>
   <transmission name="joint_tran2">
-    <type>transmission_interface/SimpleTransmission</type>
-    <joint name="arm2_joint">
-      <!-- TODO: effort is torque, maybe position is enough -->
-      <hardwareInterface>hardware_interface/EffortJointInterface</hardwareInterface>
-    </joint>
-    <actuator name="servo2">
-      <!-- TODO: effort is torque, maybe position is enough -->
-      <hardwareInterface>hardware_interface/EffortJointInterface</hardwareInterface>
-      <mechanicalReduction>1</mechanicalReduction>
-    </actuator>
+      <type>transmission_interface/SimpleTransmission</type>
+      <joint name="arm2_joint">
+        <!-- TODO: effort is torque, maybe position is enough -->
+        <hardwareInterface>hardware_interface/EffortJointInterface</hardwareInterface>
+      </joint>
+      <actuator name="servo2">
+        <!-- TODO: effort is torque, maybe position is enough -->
+        <hardwareInterface>hardware_interface/EffortJointInterface</hardwareInterface>
+        <mechanicalReduction>1</mechanicalReduction>
+      </actuator>
   </transmission>
   <joint name="arm3_joint" type="revolute">
-    <limit lower="${-pi/3}" upper="${pi/3}" effort="10.0" velocity="0.5" />
+    <limit lower="${-pi/3}" upper="${pi/3}" effort="1.0" velocity="0.5" />
     <parent link="main_body" />
     <child link="arm3_link" />
-    <origin xyz="0.03 0.03 0" rpy="0 0 ${ pi / 4}" />
+    <origin xyz="0.03015 0.03015 0.06938" rpy="0 0 ${ pi / 4}" />
     <axis xyz="0 0 1" />
     <dynamics damping="0.9" friction="0.05" />
   </joint>
   <link name="arm3_link">
-    <origin xyz="0 0 0" rpy="0 0 0" />
-    <inertial>
-      <origin xyz="${0.21 / 2 - 0.004} 0 0" rpy="0 0 0" />
-      <mass value="0.200" />
+    <inertial>
+      <origin xyz="0.138 0 -0.00104" rpy="0 0 0" />
+      <mass value="0.191" />
       <inertia
         ixx="0.001804" iyy="0.017972" izz="0.019248"
-        ixy="0.000021" ixz="0.000372" iyz="0.000000" />
-    </inertial>
-    <visual>
-      <origin xyz="${0.21 / 2 - 0.004} 0 0" rpy="0 0 0" />
-      <geometry>
-        <box size="0.21 0.015 0.005" />
+        ixy="0.000021" ixz="0.000372" iyz="0.000000"/>
+    </inertial>
+    <visual>
+      <origin xyz="0.138 0 -0.00104" rpy="0 0 0" />
+      <geometry>
+        <mesh filename="package://kinikun/urdf/mesh/kinikun2/arm.dae" />
       </geometry>
     </visual>
@@ -271,5 +271,5 @@
     <parent link="arm3_link" />
     <child link="thrust3" />
-    <origin xyz="0.19 0 0 " rpy="0 0 0" />
+    <origin xyz="0.179 0 0.0209" rpy="0 0 0" />
     <axis xyz="0 0 -1" />
     <limit effort="100" lower="${min_force}" upper="${max_force}" velocity="0.5" />
@@ -292,5 +292,5 @@
     </visual>
   </link>
-  <xacro:damping_factor link="thrust3" />
+  <xacro:damping_factor link ="thrust3"/>
   <transmission name="rotor_tran3">
     <type>transmission_interface/SimpleTransmission</type>
@@ -305,37 +305,36 @@
     </actuator>
   </transmission>
-  <transmission name="joint_tran3">
-    <type>transmission_interface/SimpleTransmission</type>
-    <joint name="arm3_joint">
-      <!-- TODO: effort is torque, maybe position is enough -->
-      <hardwareInterface>hardware_interface/EffortJointInterface</hardwareInterface>
-    </joint>
-    <actuator name="servo3">
-      <!-- TODO: effort is torque, maybe position is enough -->
-      <hardwareInterface>hardware_interface/EffortJointInterface</hardwareInterface>
-      <mechanicalReduction>1</mechanicalReduction>
-    </actuator>
-  </transmission>
-  <joint name="arm4_joint" type="fixed">
-    <!-- <limit lower="${-pi/4}" upper="${pi/4}" effort="10.0" velocity="0.5"/> -->
+      <transmission name="joint_tran3">
+      <type>transmission_interface/SimpleTransmission</type>
+      <joint name="arm3_joint">
+        <!-- TODO: effort is torque, maybe position is enough -->
+        <hardwareInterface>hardware_interface/EffortJointInterface</hardwareInterface>
+      </joint>
+      <actuator name="servo3">
+        <!-- TODO: effort is torque, maybe position is enough -->
+        <hardwareInterface>hardware_interface/EffortJointInterface</hardwareInterface>
+        <mechanicalReduction>1</mechanicalReduction>
+      </actuator>
+  </transmission>
+  <joint name="arm4_joint" type="revolute">
+    <limit lower="${-pi/4}" upper="${pi/4}" effort="1.0" velocity="0.5"/>
     <parent link="main_body" />
     <child link="arm4_link" />
-    <origin xyz="-0.03 0.03 0" rpy="0 0 ${3* pi / 4}" />
+    <origin xyz="-0.03015 0.03015 0.06938" rpy="0 0 ${pi * 3 / 4}" />
     <axis xyz="0 0 1" />
     <dynamics damping="0.9" friction="0.05" />
   </joint>
   <link name="arm4_link">
-    <origin xyz="0 0 0" rpy="0 0 0" />
-    <inertial>
-      <origin xyz="${0.21 / 2 - 0.004} 0 0" rpy="0 0 0" />
-      <mass value="0.12" />
+    <inertial>
+      <origin xyz="0.138 0 -0.00104" rpy="0 0 0" />
+      <mass value="0.191" />
       <inertia
         ixx="0.001804" iyy="0.017972" izz="0.019248"
-        ixy="0.000021" ixz="0.000372" iyz="0.000000" />
-    </inertial>
-    <visual>
-      <origin xyz="${0.21 / 2 - 0.004} 0 0" rpy="0 0 0" />
-      <geometry>
-        <box size="0.21 0.015 0.005" />
+        ixy="0.000021" ixz="0.000372" iyz="0.000000"/>
+    </inertial>
+    <visual>
+      <origin xyz="0.138 0 -0.00104" rpy="0 0 0" />
+      <geometry>
+        <mesh filename="package://kinikun/urdf/mesh/kinikun2/arm.dae" />
       </geometry>
     </visual>
@@ -344,5 +343,5 @@
     <parent link="arm4_link" />
     <child link="thrust4" />
-    <origin xyz="0.19 0 0 " rpy="0 0 0" />
+    <origin xyz="0.179 0 0.0209" rpy="0 0 0" />
     <axis xyz="0 0 1" />
     <limit effort="100" lower="${min_force}" upper="${max_force}" velocity="0.5" />
@@ -365,5 +364,5 @@
     </visual>
   </link>
-  <xacro:damping_factor link="thrust4" />
+  <xacro:damping_factor link ="thrust4"/>
   <transmission name="rotor_tran4">
     <type>transmission_interface/SimpleTransmission</type>
@@ -378,3 +377,15 @@
     </actuator>
   </transmission>
+      <transmission name="joint_tran4">
+      <type>transmission_interface/SimpleTransmission</type>
+      <joint name="arm4_joint">
+        <!-- TODO: effort is torque, maybe position is enough -->
+        <hardwareInterface>hardware_interface/EffortJointInterface</hardwareInterface>
+      </joint>
+      <actuator name="servo4">
+        <!-- TODO: effort is torque, maybe position is enough -->
+        <hardwareInterface>hardware_interface/EffortJointInterface</hardwareInterface>
+        <mechanicalReduction>1</mechanicalReduction>
+      </actuator>
+  </transmission>
 </robot>
