Commit message: [kinikun] add script for four mocap

File: robots/kinikun/urdf/robot.gazebo.xacro (robot description, xacro)
@@ -4,5 +4,5 @@
   <xacro:arg name="robot_name" default="kinikun" />
   <!-- robot urdf -->
-  <xacro:include filename="$(find kinikun)/urdf/robot2.urdf.xacro" />
+  <xacro:include filename="$(find kinikun)/urdf/robot.urdf.xacro" />
   <!-- gazebo plugin for default controller and sensors -->
   <xacro:include filename="$(find aerial_robot_simulation)/xacro/spinal.gazebo.xacro" />

File: robots/kinikun/urdf/robot.urdf.xacro (robot description, xacro)
@@ -58,21 +58,21 @@
   <link name="main_body">
     <inertial>
-      <mass value="0.210" />
-      <origin xyz="0 0 0.018" rpy="0 0 0" />
-      <inertia
-        ixx="0.000096398" ixy="0" ixz="0"
-        iyy="0.000098683" iyz="0"
-        izz="0.000157235" />
-    </inertial>
-    <visual>
-      <origin rpy="0 0 0" xyz="0 0 0" />
-      <geometry>
-        <mesh filename="package://kinikun/urdf/mesh/kinikun/kinikun_main_body.dae" />
+      <mass value="0.239" />
+      <origin xyz="0 0 0.064" rpy="0 0 0" />
+      <inertia
+        ixx="0.0021" ixy="0" ixz="0"
+        iyy="0.0015" iyz="0"
+        izz="0.0032"/>
+    </inertial>
+    <visual>
+      <origin rpy="0 0 0" xyz="0 0 0.080" />
+      <geometry>
+        <mesh filename="package://kinikun/urdf/mesh/kinikun2/main_body.dae" />
       </geometry>
     </visual>
     <collision>
-      <origin rpy="0 0 0" xyz="0 0 0" />
-      <geometry>
-        <box size="0.1 0.1 0.01" />
+      <origin rpy="0 0 0" xyz="0 0 0.064" />
+      <geometry>
+        <box size="0.1 0.1 0.018" />
       </geometry>
     </collision>
@@ -82,5 +82,5 @@
     <origin xyz="0 0 0" rpy="0 0 0" />
     <inertial>
-      <mass value="00" />
+      <mass value="0.0" />
       <origin xyz="0 0 0" rpy="0 0 0" />
       <inertia
@@ -101,25 +101,24 @@
     </inertial>
   </xacro:extra_module> -->
-  <joint name="arm1_joint" type="fixed">
-    <!-- <limit lower="${-pi/4}" upper="${pi/4}" effort="10.0" velocity="0.5"/> -->
+  <joint name="arm1_joint" type="revolute">
+    <limit lower="${-pi/4}" upper="${pi/4}" effort="1.0" velocity="0.5"/>
     <parent link="main_body" />
     <child link="arm1_link" />
-    <origin xyz="-0.03023 -0.03023 0.004" rpy="0 0 ${ -3*pi / 4}" />
+    <origin xyz="-0.03015 -0.03015 0.06938" rpy="0 0 ${ -3*pi / 4}" />
     <axis xyz="0 0 1" />
     <dynamics damping="0.9" friction="0.05" />
   </joint>
   <link name="arm1_link">
-    <origin xyz="0 0 0" rpy="0 0 0" />
-    <inertial>
-      <origin xyz="0.148 -0.004 0" rpy="0 0 0" />
-      <mass value="0.120" />
-      <inertia
-        ixx="0.000100424" iyy="0.000408408" izz="0.000429299"
-        ixy="0" ixz="0.00004" iyz="0" />
-    </inertial>
-    <visual>
-      <origin xyz="0 0 0" rpy="0 0 0" />
-      <geometry>
-        <mesh filename="package://kinikun/urdf/mesh/kinikun/kinikun_foot_R.dae" />
+    <inertial>
+      <origin xyz="0.138 0 -0.00104" rpy="0 0 0" />
+      <mass value="0.220" />
+      <inertia
+        ixx="0.001804" iyy="0.017972" izz="0.019248"
+        ixy="0.000021" ixz="0.000372" iyz="0.000000"/>
+    </inertial>
+    <visual>
+      <origin xyz="0.138 0 -0.00104" rpy="0 0 0" />
+      <geometry>
+        <mesh filename="package://kinikun/urdf/mesh/kinikun2/arm.dae" />
       </geometry>
     </visual>
@@ -162,26 +161,36 @@
     </actuator>
   </transmission>
+      <transmission name="joint_tran1">
+      <type>transmission_interface/SimpleTransmission</type>
+      <joint name="arm1_joint">
+        <!-- TODO: effort is torque, maybe position is enough -->
+        <hardwareInterface>hardware_interface/EffortJointInterface</hardwareInterface>
+      </joint>
+      <actuator name="servo1">
+        <!-- TODO: effort is torque, maybe position is enough -->
+        <hardwareInterface>hardware_interface/EffortJointInterface</hardwareInterface>
+        <mechanicalReduction>1</mechanicalReduction>
+      </actuator>
+  </transmission>
   <joint name="arm2_joint" type="revolute">
     <limit lower="${-pi/4}" upper="${pi/4}" effort="1.0" velocity="0.5" />
     <parent link="main_body" />
     <child link="arm2_link" />
-    <origin xyz="0.03023 -0.03023 0.004" rpy="0 0 ${- pi / 4}" />
+    <origin xyz="0.03015 -0.03015 0.06938" rpy="0 0 ${- pi / 4}" />
     <axis xyz="0 0 1" />
     <dynamics damping="0.9" friction="0.05" />
   </joint>
   <link name="arm2_link">
-    <origin xyz="0 0 0" rpy="0 0 0" />
-    <inertial>
-      <origin xyz="0.148 -0.004 0" rpy="0 0 0" />
-      <mass value="0.2" />
-      <!-- <mass value="0.157" /> -->
-      <inertia
-        ixx="0.000100425" iyy="0.000408408" izz="0.000429300"
-        ixy="0" ixz="0.00004" iyz="0" />
-    </inertial>
-    <visual>
-      <origin xyz="0 0 0" rpy="0 0 0" />
-      <geometry>
-        <mesh filename="package://kinikun/urdf/mesh/kinikun/kinikun_foot_L.dae" />
+    <inertial>
+      <origin xyz="0.138 0 -0.00104" rpy="0 0 0" />
+      <mass value="0.220" />
+      <inertia
+        ixx="0.001804" iyy="0.017972" izz="0.019248"
+        ixy="0.000021" ixz="0.000372" iyz="0.000000"/>
+    </inertial>
+    <visual>
+      <origin xyz="0.138 0 -0.00104" rpy="0 0 0" />
+      <geometry>
+        <mesh filename="package://kinikun/urdf/mesh/kinikun2/arm.dae" />
       </geometry>
     </visual>
@@ -211,5 +220,5 @@
     </visual>
   </link>
-  <xacro:damping_factor link="thrust2" />
+  <xacro:damping_factor link ="thrust2"/>
   <transmission name="rotor_tran2">
     <type>transmission_interface/SimpleTransmission</type>
@@ -225,14 +234,14 @@
   </transmission>
   <transmission name="joint_tran2">
-    <type>transmission_interface/SimpleTransmission</type>
-    <joint name="arm2_joint">
-      <!-- TODO: effort is torque, maybe position is enough -->
-      <hardwareInterface>hardware_interface/EffortJointInterface</hardwareInterface>
-    </joint>
-    <actuator name="servo2">
-      <!-- TODO: effort is torque, maybe position is enough -->
-      <hardwareInterface>hardware_interface/EffortJointInterface</hardwareInterface>
-      <mechanicalReduction>1</mechanicalReduction>
-    </actuator>
+      <type>transmission_interface/SimpleTransmission</type>
+      <joint name="arm2_joint">
+        <!-- TODO: effort is torque, maybe position is enough -->
+        <hardwareInterface>hardware_interface/EffortJointInterface</hardwareInterface>
+      </joint>
+      <actuator name="servo2">
+        <!-- TODO: effort is torque, maybe position is enough -->
+        <hardwareInterface>hardware_interface/EffortJointInterface</hardwareInterface>
+        <mechanicalReduction>1</mechanicalReduction>
+      </actuator>
   </transmission>
   <joint name="arm3_joint" type="revolute">
@@ -240,21 +249,20 @@
     <parent link="main_body" />
     <child link="arm3_link" />
-    <origin xyz="0.03023 0.03023 0.004" rpy="0 0 ${ pi / 4}" />
+    <origin xyz="0.03015 0.03015 0.06938" rpy="0 0 ${ pi / 4}" />
     <axis xyz="0 0 1" />
     <dynamics damping="0.9" friction="0.05" />
   </joint>
   <link name="arm3_link">
-    <origin xyz="0 0 0" rpy="0 0 0" />
-    <inertial>
-      <origin xyz="0.148 -0.004 0" rpy="0 0 0" />
-      <mass value="0.2" />
-      <inertia
-        ixx="0.000100424" iyy="0.000408408" izz="0.000429299"
-        ixy="0" ixz="0.00004" iyz="0" />
-    </inertial>
-    <visual>
-      <origin xyz="0 0 0" rpy="0 0 0" />
-      <geometry>
-        <mesh filename="package://kinikun/urdf/mesh/kinikun/kinikun_foot_R.dae" />
+    <inertial>
+      <origin xyz="0.138 0 -0.00104" rpy="0 0 0" />
+      <mass value="0.191" />
+      <inertia
+        ixx="0.001804" iyy="0.017972" izz="0.019248"
+        ixy="0.000021" ixz="0.000372" iyz="0.000000"/>
+    </inertial>
+    <visual>
+      <origin xyz="0.138 0 -0.00104" rpy="0 0 0" />
+      <geometry>
+        <mesh filename="package://kinikun/urdf/mesh/kinikun2/arm.dae" />
       </geometry>
     </visual>
@@ -284,5 +292,5 @@
     </visual>
   </link>
-  <xacro:damping_factor link="thrust3" />
+  <xacro:damping_factor link ="thrust3"/>
   <transmission name="rotor_tran3">
     <type>transmission_interface/SimpleTransmission</type>
@@ -297,37 +305,36 @@
     </actuator>
   </transmission>
-  <transmission name="joint_tran3">
-    <type>transmission_interface/SimpleTransmission</type>
-    <joint name="arm3_joint">
-      <!-- TODO: effort is torque, maybe position is enough -->
-      <hardwareInterface>hardware_interface/EffortJointInterface</hardwareInterface>
-    </joint>
-    <actuator name="servo3">
-      <!-- TODO: effort is torque, maybe position is enough -->
-      <hardwareInterface>hardware_interface/EffortJointInterface</hardwareInterface>
-      <mechanicalReduction>1</mechanicalReduction>
-    </actuator>
-  </transmission>
-  <joint name="arm4_joint" type="fixed">
-    <!-- <limit lower="${-pi/4}" upper="${pi/4}" effort="10.0" velocity="0.5"/> -->
+      <transmission name="joint_tran3">
+      <type>transmission_interface/SimpleTransmission</type>
+      <joint name="arm3_joint">
+        <!-- TODO: effort is torque, maybe position is enough -->
+        <hardwareInterface>hardware_interface/EffortJointInterface</hardwareInterface>
+      </joint>
+      <actuator name="servo3">
+        <!-- TODO: effort is torque, maybe position is enough -->
+        <hardwareInterface>hardware_interface/EffortJointInterface</hardwareInterface>
+        <mechanicalReduction>1</mechanicalReduction>
+      </actuator>
+  </transmission>
+  <joint name="arm4_joint" type="revolute">
+    <limit lower="${-pi/4}" upper="${pi/4}" effort="1.0" velocity="0.5"/>
     <parent link="main_body" />
     <child link="arm4_link" />
-    <origin xyz="-0.03023 0.03023 0.004" rpy="0 0 ${3* pi / 4}" />
+    <origin xyz="-0.03015 0.03015 0.06938" rpy="0 0 ${pi * 3 / 4}" />
     <axis xyz="0 0 1" />
     <dynamics damping="0.9" friction="0.05" />
   </joint>
   <link name="arm4_link">
-    <origin xyz="0 0 0" rpy="0 0 0" />
-    <inertial>
-      <origin xyz="0.148 -0.004 0" rpy="0 0 0" />
-      <mass value="0.12" />
-      <inertia
-        ixx="0.000100425" iyy="0.000408408" izz="0.000429300"
-        ixy="0" ixz="0.00004" iyz="0" />
-    </inertial>
-    <visual>
-      <origin xyz="0 0 0" rpy="0 0 0" />
-      <geometry>
-        <mesh filename="package://kinikun/urdf/mesh/kinikun/kinikun_foot_L.dae" />
+    <inertial>
+      <origin xyz="0.138 0 -0.00104" rpy="0 0 0" />
+      <mass value="0.191" />
+      <inertia
+        ixx="0.001804" iyy="0.017972" izz="0.019248"
+        ixy="0.000021" ixz="0.000372" iyz="0.000000"/>
+    </inertial>
+    <visual>
+      <origin xyz="0.138 0 -0.00104" rpy="0 0 0" />
+      <geometry>
+        <mesh filename="package://kinikun/urdf/mesh/kinikun2/arm.dae" />
       </geometry>
     </visual>
@@ -357,5 +364,5 @@
     </visual>
   </link>
-  <xacro:damping_factor link="thrust4" />
+  <xacro:damping_factor link ="thrust4"/>
   <transmission name="rotor_tran4">
     <type>transmission_interface/SimpleTransmission</type>
@@ -370,90 +377,15 @@
     </actuator>
   </transmission>
-  <joint name="arm2_dummy_joint_1" type="revolute">
-    <parent link="arm2_link" />
-    <child link="dummy_gripper_1" />
-    <origin xyz="0.2 0.02 0" rpy="0 0 0" /> <!-- 位置を調整 -->
-    <axis xyz="1 0 0"/>
-    <limit lower="0" upper="0.01" effort="0" velocity="0" />
-    <dynamics damping="0.2" friction="0.02" />
-  </joint>
-  <link name="dummy_gripper_1">
-    <inertial>
-        <mass value="0.00001" />
-        <origin xyz="0 0 0" rpy="0 0 0" />
-        <inertia
-          ixx="0.000001" ixy="0.0" ixz="0.0"
-          iyy="0.000001" iyz="0.0" izz="0.000002" />
-    </inertial>
-    <visual>
-      <origin xyz="0 0 0" rpy="0.0 0 0"/>
-      <geometry>
-        <box size="0.01 0.01 0.01"/>
-      </geometry>
-    </visual>
-  </link>
-  <joint name="arm2_dummy_joint_2" type="revolute">
-    <parent link="arm2_link" />
-    <child link="dummy_gripper_2" />
-    <origin xyz="0.2 -0.02 0" rpy="0 0 0" /> <!-- 位置を調整 -->
-    <axis xyz="1 0 0"/>
-    <limit lower="0" upper="0.01" effort="0" velocity="0" />
-    <dynamics damping="0.2" friction="0.02" />
-  </joint>
-  <link name="dummy_gripper_2">
-    <inertial>
-        <mass value="0.00001" />
-        <origin xyz="0 0 0" rpy="0 0 0" />
-        <inertia ixx="0.000001" ixy="0.0" ixz="0.0" iyy="0.000001" iyz="0.0" izz="0.000002" />
-    </inertial>
-    <visual>
-      <origin xyz="0 0 0" rpy="0.0 0 0"/>
-      <geometry>
-        <box size="0.01 0.01 0.01"/>
-      </geometry>
-    </visual>
-  </link>
-<!-- arm3_linkの先端にダミーリンクを追加 -->
-  <joint name="arm3_dummy_joint_1" type="revolute">
-    <parent link="arm3_link" />
-    <child link="dummy_gripper_3" />
-    <origin xyz="0.2 0.02 0" rpy="0 0 0" /> <!-- 位置を調整 -->
-    <axis xyz="1 0 0"/>
-    <limit lower="0" upper="0.01" effort="0" velocity="0" />
-    <dynamics damping="0.2" friction="0.02" />
-  </joint>
-  <link name="dummy_gripper_3">
-    <inertial>
-        <mass value="0.00001" />
-        <origin xyz="0 0 0" rpy="0 0 0" />
-        <inertia ixx="0.000001" ixy="0.0" ixz="0.0" iyy="0.000001" iyz="0.0" izz="0.000002" />
-    </inertial>
-    <visual>
-      <origin xyz="0 0 0" rpy="0.0 0 0"/>
-      <geometry>
-        <box size="0.01 0.01 0.01"/>
-      </geometry>
-    </visual>
-  </link>
-  <joint name="arm3_dummy_joint_2" type="revolute">
-    <parent link="arm3_link" />
-    <child link="dummy_gripper_4" />
-    <origin xyz="0.2 -0.02 0" rpy="0 0 0" /> <!-- 位置を調整 -->
-    <axis xyz="1 0 0"/>
-    <limit lower="0" upper="0.01" effort="0" velocity="0" />
-    <dynamics damping="0.2" friction="0.02" />
-  </joint>
-  <link name="dummy_gripper_4">
-    <inertial>
-        <mass value="0.00001" />
-        <origin xyz="0 0 0" rpy="0 0 0" />
-        <inertia ixx="0.000001" ixy="0.0" ixz="0.0" iyy="0.000001" iyz="0.0" izz="0.000002" />
-    </inertial>
-    <visual>
-      <origin xyz="0 0 0" rpy="0.0 0 0"/>
-      <geometry>
-        <box size="0.01 0.01 0.01"/>
-      </geometry>
-    </visual>
-  </link>
+      <transmission name="joint_tran4">
+      <type>transmission_interface/SimpleTransmission</type>
+      <joint name="arm4_joint">
+        <!-- TODO: effort is torque, maybe position is enough -->
+        <hardwareInterface>hardware_interface/EffortJointInterface</hardwareInterface>
+      </joint>
+      <actuator name="servo4">
+        <!-- TODO: effort is torque, maybe position is enough -->
+        <hardwareInterface>hardware_interface/EffortJointInterface</hardwareInterface>
+        <mechanicalReduction>1</mechanicalReduction>
+      </actuator>
+  </transmission>
 </robot>
