Commit message: [kinikun]Add urdf file for down rotor.

File: robots/kinikun/urdf/robot_down.urdf.xacro (robot description, xacro)
@@ -111,5 +111,5 @@
   <link name="arm1_link">
     <inertial>
-      <origin xyz="0.138 0 0.00104" rpy="0 0 0" />
+      <origin xyz="0.12795 -0 -0.00372" rpy="0 0 0" />
       <mass value="0.191" />
       <inertia
@@ -118,7 +118,7 @@
     </inertial>
     <visual>
-      <origin xyz="0.138 0 0.00104" rpy="0 0 0" />
-      <geometry>
-        <mesh filename="package://kinikun/urdf/mesh/kinikun2/arm.dae" />
+      <origin xyz="0.12795 0 -0.00772" rpy="0 0 0" />
+      <geometry>
+        <mesh filename="package://kinikun/urdf/mesh/kinikun2/down_arm.dae" />
       </geometry>
     </visual>
@@ -127,6 +127,6 @@
     <parent link="arm1_link" />
     <child link="thrust1" />
-    <origin xyz="0.179 0 0.0209" rpy="0 0 0" />
-    <axis xyz="0 0 -1" />
+    <origin xyz="0.1765 0 -0.034" rpy="0 0 0" />
+    <axis xyz="0 0 1" />
     <limit effort="100" lower="${min_force}" upper="${max_force}" velocity="0.5" />
   </joint>
@@ -183,5 +183,5 @@
   <link name="arm2_link">
     <inertial>
-      <origin xyz="0.138 0 0.00104" rpy="0 0 0" />
+      <origin xyz="0.12795 0 -0.00372" rpy="0 0 0" />
       <mass value="0.191" />
       <inertia
@@ -190,7 +190,7 @@
     </inertial>
     <visual>
-      <origin xyz="0.138 0 0.00104" rpy="0 0 0" />
-      <geometry>
-        <mesh filename="package://kinikun/urdf/mesh/kinikun2/arm.dae" />
+      <origin xyz="0.12795 0 -0.00372" rpy="0 0 0" />
+      <geometry>
+        <mesh filename="package://kinikun/urdf/mesh/kinikun2/down_arm.dae" />
       </geometry>
     </visual>
@@ -199,6 +199,6 @@
     <parent link="arm2_link" />
     <child link="thrust2" />
-    <origin xyz="0.179 0 0.0209" rpy="0 0 0" />
-    <axis xyz="0 0 1" />
+    <origin xyz="0.1765 0 -0.034" rpy="0 0 0" />
+    <axis xyz="0 0 -1" />
     <limit effort="100" lower="${min_force}" upper="${max_force}" velocity="0.5" />
   </joint>
@@ -255,5 +255,5 @@
   <link name="arm3_link">
     <inertial>
-      <origin xyz="0.138 0 0.00104" rpy="0 0 0" />
+      <origin xyz="0.12795 0 -0.00372" rpy="0 0 0" />
       <mass value="0.191" />
       <inertia
@@ -262,7 +262,7 @@
     </inertial>
     <visual>
-      <origin xyz="0.138 0 0.00104" rpy="0 0 0" />
-      <geometry>
-        <mesh filename="package://kinikun/urdf/mesh/kinikun2/arm.dae" />
+      <origin xyz="0.12795 0 -0.00372" rpy="0 0 0" />
+      <geometry>
+        <mesh filename="package://kinikun/urdf/mesh/kinikun2/down_arm.dae" />
       </geometry>
     </visual>
@@ -271,6 +271,6 @@
     <parent link="arm3_link" />
     <child link="thrust3" />
-    <origin xyz="0.179 0 0.0209" rpy="0 0 0" />
-    <axis xyz="0 0 -1" />
+    <origin xyz="0.1765 0 -0.034" rpy="0 0 0" />
+    <axis xyz="0 0 1" />
     <limit effort="100" lower="${min_force}" upper="${max_force}" velocity="0.5" />
   </joint>
@@ -327,5 +327,5 @@
   <link name="arm4_link">
     <inertial>
-      <origin xyz="0.138 0 0.00104" rpy="0 0 0" />
+      <origin xyz="0.12795 0 -0.00372" rpy="0 0 0" />
       <mass value="0.191" />
       <inertia
@@ -334,7 +334,7 @@
     </inertial>
     <visual>
-      <origin xyz="0.138 0 0.00104" rpy="0 0 0" />
-      <geometry>
-        <mesh filename="package://kinikun/urdf/mesh/kinikun2/arm.dae" />
+      <origin xyz="0.12795 0 -0.00372" rpy="0 0 0" />
+      <geometry>
+        <mesh filename="package://kinikun/urdf/mesh/kinikun2/down_arm.dae" />
       </geometry>
     </visual>
@@ -343,6 +343,6 @@
     <parent link="arm4_link" />
     <child link="thrust4" />
-    <origin xyz="0.179 0 0.0209" rpy="0 0 0" />
-    <axis xyz="0 0 1" />
+    <origin xyz="0.1765 0 -0.034" rpy="0 0 0" />
+    <axis xyz="0 0 -1" />
     <limit effort="100" lower="${min_force}" upper="${max_force}" velocity="0.5" />
   </joint>

Commit message: [kinikun]change robot_down.urdf

File: robots/kinikun/urdf/robot_down.urdf.xacro (robot description, xacro)
@@ -190,5 +190,5 @@
     </inertial>
     <visual>
-      <origin xyz="0.12795 0 -0.00372" rpy="0 0 0" />
+      <origin xyz="0.12795 0 -0.00772" rpy="0 0 0" />
       <geometry>
         <mesh filename="package://kinikun/urdf/mesh/kinikun2/down_arm.dae" />
@@ -262,5 +262,5 @@
     </inertial>
     <visual>
-      <origin xyz="0.12795 0 -0.00372" rpy="0 0 0" />
+      <origin xyz="0.12795 0 -0.00772" rpy="0 0 0" />
       <geometry>
         <mesh filename="package://kinikun/urdf/mesh/kinikun2/down_arm.dae" />
@@ -334,5 +334,5 @@
     </inertial>
     <visual>
-      <origin xyz="0.12795 0 -0.00372" rpy="0 0 0" />
+      <origin xyz="0.12795 0 -0.00772" rpy="0 0 0" />
       <geometry>
         <mesh filename="package://kinikun/urdf/mesh/kinikun2/down_arm.dae" />
