Commit message: add set_arm_mode.py

File: robots/kinikun/urdf/robot.urdf.xacro (robot description, xacro)
@@ -140,12 +140,12 @@
   <!-- propellers -->
   <!-- <xacro:propeller_module id = "1" x = "${-rotor_x}" y = "${-rotor_y}" z = "${rotor_z}" direction = "-1" /> -->
-  <xacro:propeller_module id = "2" x = "${rotor_x}" y = "${-rotor_y}" z = "${rotor_z}" direction = "1" />
+  <!-- <xacro:propeller_module id = "2" x = "${rotor_x}" y = "${-rotor_y}" z = "${rotor_z}" direction = "1" />
   <xacro:propeller_module id = "3" x = "${rotor_x}" y = "${rotor_y}" z = "${rotor_z}" direction = "-1" />
-  <xacro:propeller_module id = "4" x = "${-rotor_x}" y = "${rotor_y}" z = "${rotor_z}"  direction = "1" />
-  <joint name="arm1_joint" type="revolute">
+  <xacro:propeller_module id = "4" x = "${-rotor_x}" y = "${rotor_y}" z = "${rotor_z}"  direction = "1" /> -->
+ <joint name="arm1_joint" type="revolute">
     <limit lower="${-pi/4}" upper="${pi/4}" effort="10.0" velocity="0.5"/>
     <parent link="main_body"/>
     <child link="arm1_link"/>
-    <origin xyz="-0.1 -0.1 0" rpy="0 0 ${-3 * pi / 4}"/>
+    <origin xyz="-0.03 -0.03 0" rpy="0 0 ${ -3*pi / 4}"/>
     <axis xyz="0 0 1"/>
     <dynamics damping="0.9" friction="0.05"/>
@@ -154,14 +154,14 @@
     <origin xyz="0 0 0" rpy="0 0 0"/>
     <inertial>
-      <origin xyz="${0.3 / 2 - 0.04} 0 0" rpy="0 0 0"/>
+      <origin xyz="${0.19 / 2 - 0.004} 0 0" rpy="0 0 0"/>
       <mass value="0.1"/>
       <inertia
-    	  ixx="0.001804" iyy="0.017972" izz="0.019248"
-    	  ixy="0.000021" ixz="0.000372" iyz="0.000000"/>
+        ixx="0.001804" iyy="0.017972" izz="0.019248"
+        ixy="0.000021" ixz="0.000372" iyz="0.000000"/>
     </inertial>
     <visual>
-      <origin xyz="${0.3 / 2 - 0.04} 0 0" rpy="0 0 0"/>
-      <geometry>
-	<box size="0.3 0.04 0.01"/>
+      <origin xyz="${0.19 / 2 - 0.004} 0 0" rpy="0 0 0"/>
+      <geometry>
+  <box size="0.19 0.015 0.005"/>
       </geometry>
     </visual>
@@ -170,5 +170,5 @@
    <parent link="arm1_link"/>
    <child link="thrust1"/>
-   <origin xyz="0.25 0 0 " rpy="0 0 0"/>
+   <origin xyz="0.175 0 0 " rpy="0 0 0"/>
    <axis xyz="0 0 -1"/>
    <limit effort="100" lower="${min_force}" upper="${max_force}" velocity="0.5"/>
@@ -216,3 +216,186 @@
         </actuator>
     </transmission>
+<joint name="arm2_joint" type="fixed">
+    <!-- <limit lower="${-pi/4}" upper="${pi/4}" effort="10.0" velocity="0.5"/> -->
+    <parent link="main_body"/>
+    <child link="arm2_link"/>
+    <origin xyz="0.03 -0.03 0" rpy="0 0 ${- pi / 4}"/>
+    <axis xyz="0 0 1"/>
+    <dynamics damping="0.9" friction="0.05"/>
+  </joint>
+  <link name="arm2_link">
+    <origin xyz="0 0 0" rpy="0 0 0"/>
+    <inertial>
+      <origin xyz="${0.19 / 2 - 0.004} 0 0" rpy="0 0 0"/>
+      <mass value="0.1"/>
+      <inertia
+        ixx="0.001804" iyy="0.017972" izz="0.019248"
+        ixy="0.000021" ixz="0.000372" iyz="0.000000"/>
+    </inertial>
+    <visual>
+      <origin xyz="${0.19 / 2 - 0.004} 0 0" rpy="0 0 0"/>
+      <geometry>
+  <box size="0.19 0.015 0.005"/>
+      </geometry>
+    </visual>
+  </link>
+ <joint name="rotor2" type="continuous">
+   <parent link="arm2_link"/>
+   <child link="thrust2"/>
+   <origin xyz="0.175 0 0 " rpy="0 0 0"/>
+   <axis xyz="0 0 1"/>
+   <limit effort="100" lower="${min_force}" upper="${max_force}" velocity="0.5"/>
+  </joint>
+  <link name="thrust2">
+      <!-- visual & collisiont -->
+      <inertial>
+        <origin xyz="0 0 0" rpy="0 0 0"/>
+        <mass value="0.0091"/>
+        <inertia
+            ixx="0.00000807" ixy="0.0" ixz="0.0"
+            iyy="0.00000807" iyz="0.0"
+            izz="0.00001612"/>
+      </inertial>
+      <visual>
+        <origin rpy="0 0 0" xyz="0 0 0"/>
+        <geometry>
+          <mesh filename="package://kinikun/urdf/mesh/prop_5inch.dae" />
+        </geometry>
+      </visual>
+    </link>
+    <xacro:damping_factor link ="thrust2"/>
+    <transmission name="rotor_tran2">
+      <type>transmission_interface/SimpleTransmission</type>
+      <joint name="rotor2">
+        <!-- TODO: effort is torque, maybe position is enough -->
+        <hardwareInterface>RotorInterface</hardwareInterface>
+      </joint>
+      <actuator name="rotor2">
+        <!-- TODO: effort is torque, maybe position is enough -->
+        <hardwareInterface>RotorInterface</hardwareInterface>
+        <mechanicalReduction>1</mechanicalReduction>
+      </actuator>
+    </transmission>
+ <joint name="arm3_joint" type="fixed">
+    <!-- <limit lower="${-pi/4}" upper="${pi/4}" effort="10.0" velocity="0.5"/> -->
+    <parent link="main_body"/>
+    <child link="arm3_link"/>
+    <origin xyz="0.03 0.03 0" rpy="0 0 ${ pi / 4}"/>
+    <axis xyz="0 0 1"/>
+    <dynamics damping="0.9" friction="0.05"/>
+  </joint>
+  <link name="arm3_link">
+    <origin xyz="0 0 0" rpy="0 0 0"/>
+    <inertial>
+      <origin xyz="${0.19 / 2 - 0.004} 0 0" rpy="0 0 0"/>
+      <mass value="0.1"/>
+      <inertia
+        ixx="0.001804" iyy="0.017972" izz="0.019248"
+        ixy="0.000021" ixz="0.000372" iyz="0.000000"/>
+    </inertial>
+    <visual>
+      <origin xyz="${0.19 / 2 - 0.004} 0 0" rpy="0 0 0"/>
+      <geometry>
+  <box size="0.19 0.015 0.005"/>
+      </geometry>
+    </visual>
+  </link>
+ <joint name="rotor3" type="continuous">
+   <parent link="arm3_link"/>
+   <child link="thrust3"/>
+   <origin xyz="0.175 0 0 " rpy="0 0 0"/>
+   <axis xyz="0 0 -1"/>
+   <limit effort="100" lower="${min_force}" upper="${max_force}" velocity="0.5"/>
+  </joint>
+  <link name="thrust3">
+      <!-- visual & collisiont -->
+      <inertial>
+        <origin xyz="0 0 0" rpy="0 0 0"/>
+        <mass value="0.0091"/>
+        <inertia
+            ixx="0.00000807" ixy="0.0" ixz="0.0"
+            iyy="0.00000807" iyz="0.0"
+            izz="0.00001612"/>
+      </inertial>
+      <visual>
+        <origin rpy="0 0 0" xyz="0 0 0"/>
+        <geometry>
+          <mesh filename="package://kinikun/urdf/mesh/prop_5inch.dae" />
+        </geometry>
+      </visual>
+    </link>
+    <xacro:damping_factor link ="thrust3"/>
+    <transmission name="rotor_tran3">
+      <type>transmission_interface/SimpleTransmission</type>
+      <joint name="rotor3">
+        <!-- TODO: effort is torque, maybe position is enough -->
+        <hardwareInterface>RotorInterface</hardwareInterface>
+      </joint>
+      <actuator name="rotor3">
+        <!-- TODO: effort is torque, maybe position is enough -->
+        <hardwareInterface>RotorInterface</hardwareInterface>
+        <mechanicalReduction>1</mechanicalReduction>
+      </actuator>
+    </transmission>
+  <joint name="arm4_joint" type="fixed">
+    <!-- <limit lower="${-pi/4}" upper="${pi/4}" effort="10.0" velocity="0.5"/> -->
+    <parent link="main_body"/>
+    <child link="arm4_link"/>
+    <origin xyz="-0.03 0.03 0" rpy="0 0 ${3* pi / 4}"/>
+    <axis xyz="0 0 1"/>
+    <dynamics damping="0.9" friction="0.05"/>
+  </joint>
+  <link name="arm4_link">
+    <origin xyz="0 0 0" rpy="0 0 0"/>
+    <inertial>
+      <origin xyz="${0.19 / 2 - 0.004} 0 0" rpy="0 0 0"/>
+      <mass value="0.1"/>
+      <inertia
+        ixx="0.001804" iyy="0.017972" izz="0.019248"
+        ixy="0.000021" ixz="0.000372" iyz="0.000000"/>
+    </inertial>
+    <visual>
+      <origin xyz="${0.19 / 2 - 0.004} 0 0" rpy="0 0 0"/>
+      <geometry>
+  <box size="0.19 0.015 0.005"/>
+      </geometry>
+    </visual>
+  </link>
+ <joint name="rotor4" type="continuous">
+   <parent link="arm4_link"/>
+   <child link="thrust4"/>
+   <origin xyz="0.175 0 0 " rpy="0 0 0"/>
+   <axis xyz="0 0 1"/>
+   <limit effort="100" lower="${min_force}" upper="${max_force}" velocity="0.5"/>
+  </joint>
+  <link name="thrust4">
+      <!-- visual & collisiont -->
+      <inertial>
+        <origin xyz="0 0 0" rpy="0 0 0"/>
+        <mass value="0.0091"/>
+        <inertia
+            ixx="0.00000807" ixy="0.0" ixz="0.0"
+            iyy="0.00000807" iyz="0.0"
+            izz="0.00001612"/>
+      </inertial>
+      <visual>
+        <origin rpy="0 0 0" xyz="0 0 0"/>
+        <geometry>
+          <mesh filename="package://kinikun/urdf/mesh/prop_5inch.dae" />
+        </geometry>
+      </visual>
+    </link>
+    <xacro:damping_factor link ="thrust4"/>
+    <transmission name="rotor_tran4">
+      <type>transmission_interface/SimpleTransmission</type>
+      <joint name="rotor4">
+        <!-- TODO: effort is torque, maybe position is enough -->
+        <hardwareInterface>RotorInterface</hardwareInterface>
+      </joint>
+      <actuator name="rotor4">
+        <!-- TODO: effort is torque, maybe position is enough -->
+        <hardwareInterface>RotorInterface</hardwareInterface>
+        <mechanicalReduction>1</mechanicalReduction>
+      </actuator>
+    </transmission>
 </robot>

Commit message: [kinikun] change arm_joint1 to arm_joint3

File: robots/kinikun/urdf/robot.urdf.xacro (robot description, xacro)
@@ -143,6 +143,6 @@
   <xacro:propeller_module id = "3" x = "${rotor_x}" y = "${rotor_y}" z = "${rotor_z}" direction = "-1" />
   <xacro:propeller_module id = "4" x = "${-rotor_x}" y = "${rotor_y}" z = "${rotor_z}"  direction = "1" /> -->
- <joint name="arm1_joint" type="revolute">
-    <limit lower="${-pi/4}" upper="${pi/4}" effort="10.0" velocity="0.5"/>
+ <joint name="arm1_joint" type="fixed">
+    <!-- <limit lower="${-pi/4}" upper="${pi/4}" effort="10.0" velocity="0.5"/> -->
     <parent link="main_body"/>
     <child link="arm1_link"/>
@@ -204,16 +204,4 @@
       </actuator>
     </transmission>
-    <transmission name="joint_tran1">
-        <type>transmission_interface/SimpleTransmission</type>
-        <joint name="arm1_joint">
-          <!-- TODO: effort is torque, maybe position is enough -->
-          <hardwareInterface>hardware_interface/EffortJointInterface</hardwareInterface>
-        </joint>
-        <actuator name="servo1">
-          <!-- TODO: effort is torque, maybe position is enough -->
-          <hardwareInterface>hardware_interface/EffortJointInterface</hardwareInterface>
-          <mechanicalReduction>1</mechanicalReduction>
-        </actuator>
-    </transmission>
 <joint name="arm2_joint" type="fixed">
     <!-- <limit lower="${-pi/4}" upper="${pi/4}" effort="10.0" velocity="0.5"/> -->
@@ -277,6 +265,6 @@
       </actuator>
     </transmission>
- <joint name="arm3_joint" type="fixed">
-    <!-- <limit lower="${-pi/4}" upper="${pi/4}" effort="10.0" velocity="0.5"/> -->
+ <joint name="arm3_joint" type="revolute">
+    <limit lower="${-pi/4}" upper="${pi/4}" effort="10.0" velocity="0.5"/>
     <parent link="main_body"/>
     <child link="arm3_link"/>
@@ -338,4 +326,16 @@
       </actuator>
     </transmission>
+        <transmission name="joint_tran3">
+        <type>transmission_interface/SimpleTransmission</type>
+        <joint name="arm3_joint">
+          <!-- TODO: effort is torque, maybe position is enough -->
+          <hardwareInterface>hardware_interface/EffortJointInterface</hardwareInterface>
+        </joint>
+        <actuator name="servo3">
+          <!-- TODO: effort is torque, maybe position is enough -->
+          <hardwareInterface>hardware_interface/EffortJointInterface</hardwareInterface>
+          <mechanicalReduction>1</mechanicalReduction>
+        </actuator>
+    </transmission>
   <joint name="arm4_joint" type="fixed">
     <!-- <limit lower="${-pi/4}" upper="${pi/4}" effort="10.0" velocity="0.5"/> -->

Commit message: Mocap_expriment_succes

File: robots/kinikun/urdf/robot.urdf.xacro (robot description, xacro)
@@ -154,5 +154,5 @@
     <origin xyz="0 0 0" rpy="0 0 0"/>
     <inertial>
-      <origin xyz="${0.19 / 2 - 0.004} 0 0" rpy="0 0 0"/>
+      <origin xyz="${0.21 / 2 - 0.004} 0 0" rpy="0 0 0"/>
       <mass value="0.1"/>
       <inertia
@@ -161,7 +161,7 @@
     </inertial>
     <visual>
-      <origin xyz="${0.19 / 2 - 0.004} 0 0" rpy="0 0 0"/>
-      <geometry>
-  <box size="0.19 0.015 0.005"/>
+      <origin xyz="${0.21 / 2 - 0.004} 0 0" rpy="0 0 0"/>
+      <geometry>
+  <box size="0.21 0.015 0.005"/>
       </geometry>
     </visual>
@@ -170,5 +170,5 @@
    <parent link="arm1_link"/>
    <child link="thrust1"/>
-   <origin xyz="0.175 0 0 " rpy="0 0 0"/>
+   <origin xyz="0.19 0 0 " rpy="0 0 0"/>
    <axis xyz="0 0 -1"/>
    <limit effort="100" lower="${min_force}" upper="${max_force}" velocity="0.5"/>
@@ -215,5 +215,5 @@
     <origin xyz="0 0 0" rpy="0 0 0"/>
     <inertial>
-      <origin xyz="${0.19 / 2 - 0.004} 0 0" rpy="0 0 0"/>
+      <origin xyz="${0.21 / 2 - 0.004} 0 0" rpy="0 0 0"/>
       <mass value="0.1"/>
       <inertia
@@ -222,7 +222,7 @@
     </inertial>
     <visual>
-      <origin xyz="${0.19 / 2 - 0.004} 0 0" rpy="0 0 0"/>
-      <geometry>
-  <box size="0.19 0.015 0.005"/>
+      <origin xyz="${0.21 / 2 - 0.004} 0 0" rpy="0 0 0"/>
+      <geometry>
+  <box size="0.21 0.015 0.005"/>
       </geometry>
     </visual>
@@ -231,5 +231,5 @@
    <parent link="arm2_link"/>
    <child link="thrust2"/>
-   <origin xyz="0.175 0 0 " rpy="0 0 0"/>
+   <origin xyz="0.19 0 0 " rpy="0 0 0"/>
    <axis xyz="0 0 1"/>
    <limit effort="100" lower="${min_force}" upper="${max_force}" velocity="0.5"/>
@@ -266,5 +266,5 @@
     </transmission>
  <joint name="arm3_joint" type="revolute">
-    <limit lower="${-pi/4}" upper="${pi/4}" effort="10.0" velocity="0.5"/>
+    <limit lower="${-pi/3}" upper="${pi/3}" effort="10.0" velocity="0.5"/>
     <parent link="main_body"/>
     <child link="arm3_link"/>
@@ -276,5 +276,5 @@
     <origin xyz="0 0 0" rpy="0 0 0"/>
     <inertial>
-      <origin xyz="${0.19 / 2 - 0.004} 0 0" rpy="0 0 0"/>
+      <origin xyz="${0.21 / 2 - 0.004} 0 0" rpy="0 0 0"/>
       <mass value="0.1"/>
       <inertia
@@ -283,7 +283,7 @@
     </inertial>
     <visual>
-      <origin xyz="${0.19 / 2 - 0.004} 0 0" rpy="0 0 0"/>
-      <geometry>
-  <box size="0.19 0.015 0.005"/>
+      <origin xyz="${0.21 / 2 - 0.004} 0 0" rpy="0 0 0"/>
+      <geometry>
+  <box size="0.21 0.015 0.005"/>
       </geometry>
     </visual>
@@ -292,5 +292,5 @@
    <parent link="arm3_link"/>
    <child link="thrust3"/>
-   <origin xyz="0.175 0 0 " rpy="0 0 0"/>
+   <origin xyz="0.19 0 0 " rpy="0 0 0"/>
    <axis xyz="0 0 -1"/>
    <limit effort="100" lower="${min_force}" upper="${max_force}" velocity="0.5"/>
@@ -349,5 +349,5 @@
     <origin xyz="0 0 0" rpy="0 0 0"/>
     <inertial>
-      <origin xyz="${0.19 / 2 - 0.004} 0 0" rpy="0 0 0"/>
+      <origin xyz="${0.21 / 2 - 0.004} 0 0" rpy="0 0 0"/>
       <mass value="0.1"/>
       <inertia
@@ -356,7 +356,7 @@
     </inertial>
     <visual>
-      <origin xyz="${0.19 / 2 - 0.004} 0 0" rpy="0 0 0"/>
-      <geometry>
-  <box size="0.19 0.015 0.005"/>
+      <origin xyz="${0.21 / 2 - 0.004} 0 0" rpy="0 0 0"/>
+      <geometry>
+  <box size="0.21 0.015 0.005"/>
       </geometry>
     </visual>
@@ -365,5 +365,5 @@
    <parent link="arm4_link"/>
    <child link="thrust4"/>
-   <origin xyz="0.175 0 0 " rpy="0 0 0"/>
+   <origin xyz="0.19 0 0 " rpy="0 0 0"/>
    <axis xyz="0 0 1"/>
    <limit effort="100" lower="${min_force}" upper="${max_force}" velocity="0.5"/>

Commit message: [kinikun]1124_twoarm_experiment

File: robots/kinikun/urdf/robot.urdf.xacro (robot description, xacro)
@@ -204,6 +204,6 @@
       </actuator>
     </transmission>
-<joint name="arm2_joint" type="fixed">
-    <!-- <limit lower="${-pi/4}" upper="${pi/4}" effort="10.0" velocity="0.5"/> -->
+<joint name="arm2_joint" type="revolute">
+    <limit lower="${-pi/4}" upper="${pi/4}" effort="10.0" velocity="0.5"/>
     <parent link="main_body"/>
     <child link="arm2_link"/>
@@ -216,5 +216,5 @@
     <inertial>
       <origin xyz="${0.21 / 2 - 0.004} 0 0" rpy="0 0 0"/>
-      <mass value="0.1"/>
+      <mass value="0.2"/>
       <inertia
         ixx="0.001804" iyy="0.017972" izz="0.019248"
@@ -265,4 +265,16 @@
       </actuator>
     </transmission>
+        <transmission name="joint_tran2">
+        <type>transmission_interface/SimpleTransmission</type>
+        <joint name="arm2_joint">
+          <!-- TODO: effort is torque, maybe position is enough -->
+          <hardwareInterface>hardware_interface/EffortJointInterface</hardwareInterface>
+        </joint>
+        <actuator name="servo2">
+          <!-- TODO: effort is torque, maybe position is enough -->
+          <hardwareInterface>hardware_interface/EffortJointInterface</hardwareInterface>
+          <mechanicalReduction>1</mechanicalReduction>
+        </actuator>
+    </transmission>
  <joint name="arm3_joint" type="revolute">
     <limit lower="${-pi/3}" upper="${pi/3}" effort="10.0" velocity="0.5"/>
@@ -277,5 +289,5 @@
     <inertial>
       <origin xyz="${0.21 / 2 - 0.004} 0 0" rpy="0 0 0"/>
-      <mass value="0.1"/>
+      <mass value="0.2"/>
       <inertia
         ixx="0.001804" iyy="0.017972" izz="0.019248"

Commit message: [WIP][kinikun]pid_angle

File: robots/kinikun/urdf/robot.urdf.xacro (robot description, xacro)
@@ -96,5 +96,5 @@
   <link name="main_body">
     <inertial>
-      <mass value = "0.430" />
+      <mass value = "0.276" />
       <origin xyz="0 0 0.017" rpy="0 0 0"/>
       <inertia
@@ -155,5 +155,5 @@
     <inertial>
       <origin xyz="${0.21 / 2 - 0.004} 0 0" rpy="0 0 0"/>
-      <mass value="0.1"/>
+      <mass value="0.12"/>
       <inertia
         ixx="0.001804" iyy="0.017972" izz="0.019248"
@@ -216,5 +216,5 @@
     <inertial>
       <origin xyz="${0.21 / 2 - 0.004} 0 0" rpy="0 0 0"/>
-      <mass value="0.2"/>
+      <mass value="0.160"/>
       <inertia
         ixx="0.001804" iyy="0.017972" izz="0.019248"
@@ -289,5 +289,5 @@
     <inertial>
       <origin xyz="${0.21 / 2 - 0.004} 0 0" rpy="0 0 0"/>
-      <mass value="0.2"/>
+      <mass value="0.160"/>
       <inertia
         ixx="0.001804" iyy="0.017972" izz="0.019248"
@@ -362,5 +362,5 @@
     <inertial>
       <origin xyz="${0.21 / 2 - 0.004} 0 0" rpy="0 0 0"/>
-      <mass value="0.1"/>
+      <mass value="0.12"/>
       <inertia
         ixx="0.001804" iyy="0.017972" izz="0.019248"

Commit message: succes two arm experiment add pid pythonfile

File: robots/kinikun/urdf/robot.urdf.xacro (robot description, xacro)
@@ -216,5 +216,5 @@
     <inertial>
       <origin xyz="${0.21 / 2 - 0.004} 0 0" rpy="0 0 0"/>
-      <mass value="0.160"/>
+      <mass value="0.200"/>
       <inertia
         ixx="0.001804" iyy="0.017972" izz="0.019248"
@@ -289,5 +289,5 @@
     <inertial>
       <origin xyz="${0.21 / 2 - 0.004} 0 0" rpy="0 0 0"/>
-      <mass value="0.160"/>
+      <mass value="0.200"/>
       <inertia
         ixx="0.001804" iyy="0.017972" izz="0.019248"
