Commit message: [kinikun]add dae file of kinikun for urdf

File: robots/kinikun/urdf/robot.urdf.xacro (robot description, xacro)
@@ -58,15 +58,15 @@
   <link name="main_body">
     <inertial>
-      <mass value="0.276" />
-      <origin xyz="0 0 0.017" rpy="0 0 0" />
-      <inertia
-        ixx="0.0021" ixy="0" ixz="0"
-        iyy="0.0015" iyz="0"
-        izz="0.0032" />
-    </inertial>
-    <visual>
-      <origin rpy="0 0 0" xyz="0 0 0" />
-      <geometry>
-        <mesh filename="package://kinikun/urdf/mesh/main_body.dae" />
+      <mass value="0.210" />
+      <origin xyz="0 0 0.018" rpy="0 0 0" />
+      <inertia
+        ixx="0.000096398" ixy="0" ixz="0"
+        iyy="0.000098683" iyz="0"
+        izz="0.000157235" />
+    </inertial>
+    <visual>
+      <origin rpy="0 0 0" xyz="0 0 0" />
+      <geometry>
+        <mesh filename="package://kinikun/urdf/mesh/kinikun_main_body.dae" />
       </geometry>
     </visual>
@@ -74,5 +74,5 @@
       <origin rpy="0 0 0" xyz="0 0 0" />
       <geometry>
-        <box size="0.28 0.28 0.072" />
+        <box size="0.1 0.1 0.080" />
       </geometry>
     </collision>
@@ -89,5 +89,5 @@
     </inertial>
   </xacro:extra_module>
-  <!-- battery -->
+  <!-- battery
   <xacro:extra_module name="battery" parent="main_body" visible="1"
     model_url="package://kinikun/urdf/mesh/turnigy_3S_2200mAh.dae">
@@ -100,10 +100,10 @@
         iyy="0.0002" iyz="0.0" izz="0.0002" />
     </inertial>
-  </xacro:extra_module>
+  </xacro:extra_module> -->
   <joint name="arm1_joint" type="fixed">
     <!-- <limit lower="${-pi/4}" upper="${pi/4}" effort="10.0" velocity="0.5"/> -->
     <parent link="main_body" />
     <child link="arm1_link" />
-    <origin xyz="-0.03 -0.03 0" rpy="0 0 ${ -3*pi / 4}" />
+    <origin xyz="-0.03023 -0.03023 0.004" rpy="0 0 ${ -3*pi / 4}" />
     <axis xyz="0 0 1" />
     <dynamics damping="0.9" friction="0.05" />
@@ -112,14 +112,14 @@
     <origin xyz="0 0 0" rpy="0 0 0" />
     <inertial>
-      <origin xyz="${0.21 / 2 - 0.004} 0 0" rpy="0 0 0" />
-      <mass value="0.12" />
-      <inertia
-        ixx="0.001804" iyy="0.017972" izz="0.019248"
-        ixy="0.000021" ixz="0.000372" iyz="0.000000" />
-    </inertial>
-    <visual>
-      <origin xyz="${0.21 / 2 - 0.004} 0 0" rpy="0 0 0" />
-      <geometry>
-        <box size="0.21 0.015 0.005" />
+      <origin xyz="0.148 -0.004 0" rpy="0 0 0" />
+      <mass value="0.157" />
+      <inertia
+        ixx="0.000100424" iyy="0.000408408" izz="0.000429299"
+        ixy="0" ixz="0.00004" iyz="0" />
+    </inertial>
+    <visual>
+      <origin xyz="0 0 0" rpy="0 0 0" />
+      <geometry>
+        <mesh filename="package://kinikun/urdf/mesh/kinikun_foot_R.dae" />
       </geometry>
     </visual>
@@ -128,5 +128,5 @@
     <parent link="arm1_link" />
     <child link="thrust1" />
-    <origin xyz="0.19 0 0 " rpy="0 0 0" />
+    <origin xyz="0.179 0 0.0209" rpy="0 0 0" />
     <axis xyz="0 0 -1" />
     <limit effort="100" lower="${min_force}" upper="${max_force}" velocity="0.5" />
@@ -163,8 +163,8 @@
   </transmission>
   <joint name="arm2_joint" type="revolute">
-    <limit lower="${-pi/4}" upper="${pi/4}" effort="10.0" velocity="0.5" />
+    <limit lower="${-pi/4}" upper="${pi/4}" effort="1.0" velocity="0.5" />
     <parent link="main_body" />
     <child link="arm2_link" />
-    <origin xyz="0.03 -0.03 0" rpy="0 0 ${- pi / 4}" />
+    <origin xyz="0.03023 -0.03023 0.004" rpy="0 0 ${- pi / 4}" />
     <axis xyz="0 0 1" />
     <dynamics damping="0.9" friction="0.05" />
@@ -173,14 +173,14 @@
     <origin xyz="0 0 0" rpy="0 0 0" />
     <inertial>
-      <origin xyz="${0.21 / 2 - 0.004} 0 0" rpy="0 0 0" />
-      <mass value="0.200" />
-      <inertia
-        ixx="0.001804" iyy="0.017972" izz="0.019248"
-        ixy="0.000021" ixz="0.000372" iyz="0.000000" />
-    </inertial>
-    <visual>
-      <origin xyz="${0.21 / 2 - 0.004} 0 0" rpy="0 0 0" />
-      <geometry>
-        <box size="0.21 0.015 0.005" />
+      <origin xyz="0.148 -0.004 0" rpy="0 0 0" />
+      <mass value="0.157" />
+      <inertia
+        ixx="0.000100425" iyy="0.000408408" izz="0.000429300"
+        ixy="0" ixz="0.00004" iyz="0" />
+    </inertial>
+    <visual>
+      <origin xyz="0 0 0" rpy="0 0 0" />
+      <geometry>
+        <mesh filename="package://kinikun/urdf/mesh/kinikun_foot_L.dae" />
       </geometry>
     </visual>
@@ -189,5 +189,5 @@
     <parent link="arm2_link" />
     <child link="thrust2" />
-    <origin xyz="0.19 0 0 " rpy="0 0 0" />
+    <origin xyz="0.179 0 0.0209" rpy="0 0 0" />
     <axis xyz="0 0 1" />
     <limit effort="100" lower="${min_force}" upper="${max_force}" velocity="0.5" />
@@ -236,8 +236,8 @@
   </transmission>
   <joint name="arm3_joint" type="revolute">
-    <limit lower="${-pi/3}" upper="${pi/3}" effort="10.0" velocity="0.5" />
+    <limit lower="${-pi/3}" upper="${pi/3}" effort="1.0" velocity="0.5" />
     <parent link="main_body" />
     <child link="arm3_link" />
-    <origin xyz="0.03 0.03 0" rpy="0 0 ${ pi / 4}" />
+    <origin xyz="0.03023 0.03023 0.004" rpy="0 0 ${ pi / 4}" />
     <axis xyz="0 0 1" />
     <dynamics damping="0.9" friction="0.05" />
@@ -246,14 +246,14 @@
     <origin xyz="0 0 0" rpy="0 0 0" />
     <inertial>
-      <origin xyz="${0.21 / 2 - 0.004} 0 0" rpy="0 0 0" />
-      <mass value="0.200" />
-      <inertia
-        ixx="0.001804" iyy="0.017972" izz="0.019248"
-        ixy="0.000021" ixz="0.000372" iyz="0.000000" />
-    </inertial>
-    <visual>
-      <origin xyz="${0.21 / 2 - 0.004} 0 0" rpy="0 0 0" />
-      <geometry>
-        <box size="0.21 0.015 0.005" />
+      <origin xyz="0.148 -0.004 0" rpy="0 0 0" />
+      <mass value="0.157" />
+      <inertia
+        ixx="0.000100424" iyy="0.000408408" izz="0.000429299"
+        ixy="0" ixz="0.00004" iyz="0" />
+    </inertial>
+    <visual>
+      <origin xyz="0 0 0" rpy="0 0 0" />
+      <geometry>
+        <mesh filename="package://kinikun/urdf/mesh/kinikun_foot_R.dae" />
       </geometry>
     </visual>
@@ -262,5 +262,5 @@
     <parent link="arm3_link" />
     <child link="thrust3" />
-    <origin xyz="0.19 0 0 " rpy="0 0 0" />
+    <origin xyz="0.179 0 0.0209" rpy="0 0 0" />
     <axis xyz="0 0 -1" />
     <limit effort="100" lower="${min_force}" upper="${max_force}" velocity="0.5" />
@@ -312,5 +312,5 @@
     <parent link="main_body" />
     <child link="arm4_link" />
-    <origin xyz="-0.03 0.03 0" rpy="0 0 ${3* pi / 4}" />
+    <origin xyz="-0.03023 0.03023 0.004" rpy="0 0 ${3* pi / 4}" />
     <axis xyz="0 0 1" />
     <dynamics damping="0.9" friction="0.05" />
@@ -319,14 +319,14 @@
     <origin xyz="0 0 0" rpy="0 0 0" />
     <inertial>
-      <origin xyz="${0.21 / 2 - 0.004} 0 0" rpy="0 0 0" />
-      <mass value="0.12" />
-      <inertia
-        ixx="0.001804" iyy="0.017972" izz="0.019248"
-        ixy="0.000021" ixz="0.000372" iyz="0.000000" />
-    </inertial>
-    <visual>
-      <origin xyz="${0.21 / 2 - 0.004} 0 0" rpy="0 0 0" />
-      <geometry>
-        <box size="0.21 0.015 0.005" />
+      <origin xyz="0.148 -0.004 0" rpy="0 0 0" />
+      <mass value="0.157" />
+      <inertia
+        ixx="0.000100425" iyy="0.000408408" izz="0.000429300"
+        ixy="0" ixz="0.00004" iyz="0" />
+    </inertial>
+    <visual>
+      <origin xyz="0 0 0" rpy="0 0 0" />
+      <geometry>
+        <mesh filename="package://kinikun/urdf/mesh/kinikun_foot_L.dae" />
       </geometry>
     </visual>
@@ -335,5 +335,5 @@
     <parent link="arm4_link" />
     <child link="thrust4" />
-    <origin xyz="0.19 0 0 " rpy="0 0 0" />
+    <origin xyz="0.179 0 0.0209" rpy="0 0 0" />
     <axis xyz="0 0 1" />
     <limit effort="100" lower="${min_force}" upper="${max_force}" velocity="0.5" />
@@ -374,5 +374,5 @@
     <origin xyz="0.2 0.02 0" rpy="0 0 0" /> <!-- 位置を調整 -->
     <axis xyz="1 0 0"/>
-    <limit lower="0" upper="0" effort="0" velocity="0" />
+    <limit lower="0" upper="0.01" effort="0" velocity="0" />
     <dynamics damping="0.2" friction="0.02" />
   </joint>
@@ -385,10 +385,4 @@
           iyy="0.000001" iyz="0.0" izz="0.000002" />
     </inertial>
-    <collision>
-      <orgin xyz="0 0 0" rpy="0 0 0" />
-      <geometry>
-        <box size="0.01 0.01 0.01" />
-      </geometry>
-    </collision>
     <visual>
       <origin xyz="0 0 0" rpy="0.0 0 0"/>
@@ -403,5 +397,5 @@
     <origin xyz="0.2 -0.02 0" rpy="0 0 0" /> <!-- 位置を調整 -->
     <axis xyz="1 0 0"/>
-    <limit lower="0" upper="0" effort="0" velocity="0" />
+    <limit lower="0" upper="0.01" effort="0" velocity="0" />
     <dynamics damping="0.2" friction="0.02" />
   </joint>
@@ -412,10 +406,4 @@
         <inertia ixx="0.000001" ixy="0.0" ixz="0.0" iyy="0.000001" iyz="0.0" izz="0.000002" />
     </inertial>
-    <collision>
-      <orgin xyz="0 0 0" rpy="0 0 0" />
-      <geometry>
-        <box size="0.01 0.01 0.01" />
-      </geometry>
-    </collision>
     <visual>
       <origin xyz="0 0 0" rpy="0.0 0 0"/>
@@ -431,5 +419,5 @@
     <origin xyz="0.2 0.02 0" rpy="0 0 0" /> <!-- 位置を調整 -->
     <axis xyz="1 0 0"/>
-    <limit lower="0" upper="0" effort="0" velocity="0" />
+    <limit lower="0" upper="0.01" effort="0" velocity="0" />
     <dynamics damping="0.2" friction="0.02" />
   </joint>
@@ -440,10 +428,4 @@
         <inertia ixx="0.000001" ixy="0.0" ixz="0.0" iyy="0.000001" iyz="0.0" izz="0.000002" />
     </inertial>
-    <collision>
-      <orgin xyz="0 0 0" rpy="0 0 0" />
-      <geometry>
-        <box size="0.01 0.01 0.01" />
-      </geometry>
-    </collision>
     <visual>
       <origin xyz="0 0 0" rpy="0.0 0 0"/>
@@ -458,5 +440,5 @@
     <origin xyz="0.2 -0.02 0" rpy="0 0 0" /> <!-- 位置を調整 -->
     <axis xyz="1 0 0"/>
-    <limit lower="0" upper="0" effort="0" velocity="0" />
+    <limit lower="0" upper="0.01" effort="0" velocity="0" />
     <dynamics damping="0.2" friction="0.02" />
   </joint>
@@ -467,10 +449,4 @@
         <inertia ixx="0.000001" ixy="0.0" ixz="0.0" iyy="0.000001" iyz="0.0" izz="0.000002" />
     </inertial>
-    <collision>
-      <orgin xyz="0 0 0" rpy="0 0 0" />
-      <geometry>
-        <box size="0.01 0.01 0.01" />
-      </geometry>
-    </collision>
     <visual>
       <origin xyz="0 0 0" rpy="0.0 0 0"/>

Commit message: [kinikun]Add force sencor

File: robots/kinikun/urdf/robot.urdf.xacro (robot description, xacro)
@@ -74,5 +74,5 @@
       <origin rpy="0 0 0" xyz="0 0 0" />
       <geometry>
-        <box size="0.1 0.1 0.080" />
+        <box size="0.1 0.1 0.01" />
       </geometry>
     </collision>
@@ -113,5 +113,5 @@
     <inertial>
       <origin xyz="0.148 -0.004 0" rpy="0 0 0" />
-      <mass value="0.157" />
+      <mass value="0.120" />
       <inertia
         ixx="0.000100424" iyy="0.000408408" izz="0.000429299"
@@ -174,5 +174,6 @@
     <inertial>
       <origin xyz="0.148 -0.004 0" rpy="0 0 0" />
-      <mass value="0.157" />
+      <mass value="0.2" />
+      <!-- <mass value="0.157" /> -->
       <inertia
         ixx="0.000100425" iyy="0.000408408" izz="0.000429300"
@@ -247,5 +248,5 @@
     <inertial>
       <origin xyz="0.148 -0.004 0" rpy="0 0 0" />
-      <mass value="0.157" />
+      <mass value="0.2" />
       <inertia
         ixx="0.000100424" iyy="0.000408408" izz="0.000429299"
@@ -320,5 +321,5 @@
     <inertial>
       <origin xyz="0.148 -0.004 0" rpy="0 0 0" />
-      <mass value="0.157" />
+      <mass value="0.12" />
       <inertia
         ixx="0.000100425" iyy="0.000408408" izz="0.000429300"

Commit message: [kinikun] Successful flight in a model with four deformable arms

File: robots/kinikun/urdf/robot.urdf.xacro (robot description, xacro)
@@ -112,5 +112,5 @@
     <inertial>
       <origin xyz="0.138 0 -0.00104" rpy="0 0 0" />
-      <mass value="0.220" />
+      <mass value="0.191" />
       <inertia
         ixx="0.001804" iyy="0.017972" izz="0.019248"
@@ -184,5 +184,5 @@
     <inertial>
       <origin xyz="0.138 0 -0.00104" rpy="0 0 0" />
-      <mass value="0.220" />
+      <mass value="0.191" />
       <inertia
         ixx="0.001804" iyy="0.017972" izz="0.019248"

Commit message: [kinikun] change the number of encoder

File: robots/kinikun/urdf/robot.urdf.xacro (robot description, xacro)
@@ -111,5 +111,5 @@
   <link name="arm1_link">
     <inertial>
-      <origin xyz="0.138 0 0.00104" rpy="0 0 0" />
+      <origin xyz="0.12795 -0 -0.00372" rpy="0 0 0" />
       <mass value="0.191" />
       <inertia
@@ -118,7 +118,7 @@
     </inertial>
     <visual>
-      <origin xyz="0.138 0 0.00104" rpy="0 0 0" />
-      <geometry>
-        <mesh filename="package://kinikun/urdf/mesh/kinikun2/arm.dae" />
+      <origin xyz="0.12795 0 -0.00772" rpy="0 0 0" />
+      <geometry>
+        <mesh filename="package://kinikun/urdf/mesh/kinikun2/down_arm.dae" />
       </geometry>
     </visual>
@@ -127,6 +127,6 @@
     <parent link="arm1_link" />
     <child link="thrust1" />
-    <origin xyz="0.179 0 0.0209" rpy="0 0 0" />
-    <axis xyz="0 0 -1" />
+    <origin xyz="0.1765 0 -0.034" rpy="0 0 0" />
+    <axis xyz="0 0 1" />
     <limit effort="100" lower="${min_force}" upper="${max_force}" velocity="0.5" />
   </joint>
@@ -183,5 +183,5 @@
   <link name="arm2_link">
     <inertial>
-      <origin xyz="0.138 0 0.00104" rpy="0 0 0" />
+      <origin xyz="0.12795 0 -0.00372" rpy="0 0 0" />
       <mass value="0.191" />
       <inertia
@@ -190,7 +190,7 @@
     </inertial>
     <visual>
-      <origin xyz="0.138 0 0.00104" rpy="0 0 0" />
-      <geometry>
-        <mesh filename="package://kinikun/urdf/mesh/kinikun2/arm.dae" />
+      <origin xyz="0.12795 0 -0.00772" rpy="0 0 0" />
+      <geometry>
+        <mesh filename="package://kinikun/urdf/mesh/kinikun2/down_arm.dae" />
       </geometry>
     </visual>
@@ -199,6 +199,6 @@
     <parent link="arm2_link" />
     <child link="thrust2" />
-    <origin xyz="0.179 0 0.0209" rpy="0 0 0" />
-    <axis xyz="0 0 1" />
+    <origin xyz="0.1765 0 -0.034" rpy="0 0 0" />
+    <axis xyz="0 0 -1" />
     <limit effort="100" lower="${min_force}" upper="${max_force}" velocity="0.5" />
   </joint>
@@ -255,5 +255,5 @@
   <link name="arm3_link">
     <inertial>
-      <origin xyz="0.138 0 0.00104" rpy="0 0 0" />
+      <origin xyz="0.12795 0 -0.00372" rpy="0 0 0" />
       <mass value="0.191" />
       <inertia
@@ -262,7 +262,7 @@
     </inertial>
     <visual>
-      <origin xyz="0.138 0 0.00104" rpy="0 0 0" />
-      <geometry>
-        <mesh filename="package://kinikun/urdf/mesh/kinikun2/arm.dae" />
+      <origin xyz="0.12795 0 -0.00772" rpy="0 0 0" />
+      <geometry>
+        <mesh filename="package://kinikun/urdf/mesh/kinikun2/down_arm.dae" />
       </geometry>
     </visual>
@@ -271,6 +271,6 @@
     <parent link="arm3_link" />
     <child link="thrust3" />
-    <origin xyz="0.179 0 0.0209" rpy="0 0 0" />
-    <axis xyz="0 0 -1" />
+    <origin xyz="0.1765 0 -0.034" rpy="0 0 0" />
+    <axis xyz="0 0 1" />
     <limit effort="100" lower="${min_force}" upper="${max_force}" velocity="0.5" />
   </joint>
@@ -327,5 +327,5 @@
   <link name="arm4_link">
     <inertial>
-      <origin xyz="0.138 0 0.00104" rpy="0 0 0" />
+      <origin xyz="0.12795 0 -0.00372" rpy="0 0 0" />
       <mass value="0.191" />
       <inertia
@@ -334,7 +334,7 @@
     </inertial>
     <visual>
-      <origin xyz="0.138 0 0.00104" rpy="0 0 0" />
-      <geometry>
-        <mesh filename="package://kinikun/urdf/mesh/kinikun2/arm.dae" />
+      <origin xyz="0.12795 0 -0.00772" rpy="0 0 0" />
+      <geometry>
+        <mesh filename="package://kinikun/urdf/mesh/kinikun2/down_arm.dae" />
       </geometry>
     </visual>
@@ -343,6 +343,6 @@
     <parent link="arm4_link" />
     <child link="thrust4" />
-    <origin xyz="0.179 0 0.0209" rpy="0 0 0" />
-    <axis xyz="0 0 1" />
+    <origin xyz="0.1765 0 -0.034" rpy="0 0 0" />
+    <axis xyz="0 0 -1" />
     <limit effort="100" lower="${min_force}" upper="${max_force}" velocity="0.5" />
   </joint>

Commit message: [kinikun]add pair sync in presure control

File: robots/kinikun/urdf/robot.urdf.xacro (robot description, xacro)
@@ -58,5 +58,5 @@
   <link name="main_body">
     <inertial>
-      <mass value="0.239" />
+      <mass value="0.47035" />
       <origin xyz="0 0 0.06462" rpy="0 0 0" />
       <inertia
@@ -112,5 +112,5 @@
     <inertial>
       <origin xyz="0.12795 -0 -0.00372" rpy="0 0 0" />
-      <mass value="0.191" />
+      <mass value="0.128" />
       <inertia
         ixx="0.001804" iyy="0.017972" izz="0.019248"
@@ -184,5 +184,5 @@
     <inertial>
       <origin xyz="0.12795 0 -0.00372" rpy="0 0 0" />
-      <mass value="0.191" />
+      <mass value="0.128" />
       <inertia
         ixx="0.001804" iyy="0.017972" izz="0.019248"
@@ -256,5 +256,5 @@
     <inertial>
       <origin xyz="0.12795 0 -0.00372" rpy="0 0 0" />
-      <mass value="0.191" />
+      <mass value="0.128" />
       <inertia
         ixx="0.001804" iyy="0.017972" izz="0.019248"
@@ -328,5 +328,5 @@
     <inertial>
       <origin xyz="0.12795 0 -0.00372" rpy="0 0 0" />
-      <mass value="0.191" />
+      <mass value="0.128" />
       <inertia
         ixx="0.001804" iyy="0.017972" izz="0.019248"
